File: doc/pcb/OttoPi01/OttoPi01.brd (EAGLE design)
At the start: 160 x 100 mm, 16 parts

Commit message: pcb
Parts:
- added JP1: (no value), pinhead:2X20
- moved LED1 23.0 mm to (17.8, 55.9)
- moved R1 12.7 mm to (17.8, 49.5)
- moved S1 3.59 mm to (7.62, 43.2)
Connections:
- removed net 3V3@1: JP11.1, JP6.1, U$1.1
- removed net 5V0@1: DC-DC.3, U$1.2
- removed net GND@8: U$1.6
- new net N$4: AMP.2, C1.2
- new net N$5: AMP.3, C1.1
- new net N$6: DC-DC.3, JP1.2
- new net N$7: JP1.5, JP11.3, JP6.3
- net GND: now also JP1.6
- net N$2: now also JP1.3; no longer U$1.3
- net N$3: now also JP1.1, JP11.1, JP6.1; no longer JP11.3, JP6.3, U$1.5
Changed lines of the file:
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@@
 <attribute name="VALUE" x="11.43" y="36.195" size="1.27" layer="27" rot="R180"/>
 </element>
-<element name="LED1" library="led" library_urn="urn:adsk.eagle:library:259" package="LED5MM" package3d_urn="urn:adsk.eagle:package:15799/2" value="" x="40.64" y="58.42" smashed="yes">
-<attribute name="NAME" x="43.815" y="58.9534" size="1.27" layer="25" ratio="10"/>
-<attribute name="POPULARITY" value="93" x="73.66" y="22.86" size="1.778" layer="27" display="off"/>
-<attribute name="VALUE" x="43.8404" y="56.6166" size="1.27" layer="27" ratio="10"/>
+<element name="LED1" library="led" library_urn="urn:adsk.eagle:library:259" package="LED5MM" package3d_urn="urn:adsk.eagle:package:15799/2" value="" x="17.78" y="55.88" smashed="yes">
+<attribute name="NAME" x="20.955" y="56.4134" size="1.27" layer="25" ratio="10"/>
+<attribute name="POPULARITY" value="93" x="50.8" y="20.32" size="1.778" layer="27" display="off"/>
+<attribute name="VALUE" x="20.9804" y="54.0766" size="1.27" layer="27" ratio="10"/>
 </element>
-<element name="S1" library="switch" library_urn="urn:adsk.eagle:library:380" package="TL3XPO" package3d_urn="urn:adsk.eagle:package:27745/1" value="TL32PO" x="10.16" y="40.64" smashed="yes" rot="R90">
-<attribute name="NAME" x="6.985" y="35.56" size="1.778" layer="25" rot="R90"/>
-<attribute name="POPULARITY" value="2" x="48.26" y="59.69" size="1.778" layer="27" rot="R90" display="off"/>
-<attribute name="VALUE" x="15.24" y="35.56" size="1.778" layer="27" rot="R90"/>
+<element name="S1" library="switch" library_urn="urn:adsk.eagle:library:380" package="TL3XPO" package3d_urn="urn:adsk.eagle:package:27745/1" value="TL32PO" x="7.62" y="43.18" smashed="yes" rot="R90">
+<attribute name="NAME" x="4.445" y="38.1" size="1.778" layer="25" rot="R90"/>
+<attribute name="POPULARITY" value="2" x="45.72" y="62.23" size="1.778" layer="27" rot="R90" display="off"/>
+<attribute name="VALUE" x="12.7" y="38.1" size="1.778" layer="27" rot="R90"/>
 </element>
 <element name="U$1" library="RPI-Zero" package="RASPBERRYPI_BASTELSTUBE_V13_RASPI_BOARD_B+_FULL" value="RPI-ZERO" x="5.08" y="-41.91" smashed="yes"/>
-<element name="R1" library="rcl" library_urn="urn:adsk.eagle:library:334" package="0204/5" package3d_urn="urn:adsk.eagle:package:23488/1" value="" x="27.94" y="57.15" smashed="yes">
-<attribute name="NAME" x="25.9334" y="58.3184" size="0.9906" layer="25" ratio="10"/>
-<attribute name="POPULARITY" value="35" x="27.94" y="57.15" size="1.778" layer="27" display="off"/>
-<attribute name="SPICEPREFIX" value="R" x="27.94" y="57.15" size="1.778" layer="27" display="off"/>
-<attribute name="VALUE" x="25.8064" y="54.8386" size="0.9906" layer="27" ratio="10"/>
+<element name="R1" library="rcl" library_urn="urn:adsk.eagle:library:334" package="0204/5" package3d_urn="urn:adsk.eagle:package:23488/1" value="" x="17.78" y="49.53" smashed="yes">
+<attribute name="NAME" x="15.7734" y="50.6984" size="0.9906" layer="25" ratio="10"/>
+<attribute name="POPULARITY" value="35" x="17.78" y="49.53" size="1.778" layer="27" display="off"/>
+<attribute name="SPICEPREFIX" value="R" x="17.78" y="49.53" size="1.778" layer="27" display="off"/>
+<attribute name="VALUE" x="15.6464" y="47.2186" size="0.9906" layer="27" ratio="10"/>
 </element>
 <element name="C1" library="rcl" library_urn="urn:adsk.eagle:library:334" package="C025-024X044" package3d_urn="urn:adsk.eagle:package:23630/1" value="" x="52.07" y="22.86" smashed="yes">
@@
 <attribute name="VALUE" x="16.51" y="32.385" size="1.27" layer="27"/>
 </element>
+<element name="JP1" library="pinhead" library_urn="urn:adsk.eagle:library:325" package="2X20" package3d_urn="urn:adsk.eagle:package:22443/2" value="" x="58.42" y="15.24" smashed="yes">
+<attribute name="NAME" x="33.02" y="18.415" size="1.27" layer="25" ratio="10"/>
+<attribute name="POPULARITY" value="12" x="58.42" y="15.24" size="1.778" layer="27" display="off"/>
+<attribute name="VALUE" x="33.02" y="10.795" size="1.27" layer="27"/>
+</element>
 </elements>
 <signals>
@@
 <contactref element="VIN" pad="1"/>
 <contactref element="S1" pad="1"/>
-<wire x1="10.16" y1="33.02" x2="10.16" y2="38.1" width="0" layer="19" extent="1-1"/>
+<wire x1="10.16" y1="33.02" x2="7.62" y2="40.64" width="0" layer="19" extent="1-1"/>
 </signal>
 <signal name="N$244">
@@
 <wire x1="35.56" y1="43.18" x2="40.64" y2="43.18" width="0" layer="19" extent="1-1"/>
 <wire x1="30.48" y1="43.18" x2="35.56" y2="43.18" width="0" layer="19" extent="1-1"/>
-<wire x1="10.16" y1="40.64" x2="30.48" y2="43.18" width="0" layer="19" extent="1-1"/>
+<wire x1="7.62" y1="43.18" x2="30.48" y2="43.18" width="0" layer="19" extent="1-1"/>
 <wire x1="10.16" y1="27.94" x2="30.48" y2="43.18" width="0" layer="19" extent="1-1"/>
-<wire x1="25.4" y1="57.15" x2="45.72" y2="43.18" width="0" layer="19" extent="1-1"/>
+<wire x1="15.24" y1="49.53" x2="45.72" y2="43.18" width="0" layer="19" extent="1-1"/>
 </signal>
 <signal name="GND">
@@
 <contactref element="SV4" pad="1"/>
 <contactref element="SV1" pad="1"/>
+<contactref element="LED1" pad="K"/>
+<contactref element="JP1" pad="6"/>
 <contactref element="JP6" pad="4"/>
 <contactref element="JP11" pad="4"/>
-<contactref element="LED1" pad="K"/>
-<wire x1="40.64" y1="45.72" x2="41.91" y2="58.42" width="0" layer="19" extent="1-1"/>
+<wire x1="40.64" y1="45.72" x2="19.05" y2="55.88" width="0" layer="19" extent="1-1"/>
 <wire x1="45.72" y1="45.72" x2="40.64" y2="45.72" width="0" layer="19" extent="1-1"/>
 <wire x1="35.56" y1="45.72" x2="40.64" y2="45.72" width="0" layer="19" extent="1-1"/>
@@
 <wire x1="25.4" y1="40.64" x2="30.48" y2="45.72" width="0" layer="19" extent="1-1"/>
 <wire x1="25.4" y1="35.56" x2="25.4" y2="40.64" width="0" layer="19" extent="1-1"/>
-<wire x1="7.62" y1="27.94" x2="25.4" y2="35.56" width="0" layer="19" extent="1-1"/>
-<wire x1="7.62" y1="33.02" x2="7.62" y2="27.94" width="0" layer="19" extent="1-1"/>
-</signal>
-<signal name="5V0@1">
-<contactref element="DC-DC" pad="3"/>
-<contactref element="U$1" pad="2"/>
-<wire x1="13.45" y1="-14.14" x2="5.08" y2="27.94" width="0" layer="19" extent="1-1"/>
-</signal>
-<signal name="GND@8">
-<contactref element="U$1" pad="6"/>
+<wire x1="7.62" y1="33.02" x2="25.4" y2="35.56" width="0" layer="19" extent="1-1"/>
+<wire x1="7.62" y1="27.94" x2="7.62" y2="33.02" width="0" layer="19" extent="1-1"/>
+<wire x1="39.37" y1="16.51" x2="7.62" y2="27.94" width="0" layer="19" extent="1-1"/>
 </signal>
 <signal name="N$248">
@@
 <wire x1="53.34" y1="43.18" x2="53.34" y2="33.02" width="0" layer="19" extent="1-1"/>
 </signal>
+<signal name="N$1">
+<contactref element="R1" pad="2"/>
+<contactref element="LED1" pad="A"/>
+<wire x1="16.51" y1="55.88" x2="20.32" y2="49.53" width="0" layer="19" extent="1-1"/>
+</signal>
+<signal name="N$4">
+<contactref element="AMP" pad="2"/>
+<contactref element="C1" pad="2"/>
+<wire x1="53.34" y1="22.86" x2="50.8" y2="25.4" width="0" layer="19" extent="1-1"/>
+</signal>
+<signal name="N$5">
+<contactref element="AMP" pad="3"/>
+<contactref element="C1" pad="1"/>
+<wire x1="50.8" y1="22.86" x2="53.34" y2="25.4" width="0" layer="19" extent="1-1"/>
+</signal>
 <signal name="N$2">
 <contactref element="JP6" pad="2"/>
 <contactref element="JP11" pad="2"/>
-<contactref element="U$1" pad="3"/>
+<contactref element="JP1" pad="3"/>
 <wire x1="20.32" y1="35.56" x2="20.32" y2="40.64" width="0" layer="19" extent="1-1"/>
-<wire x1="15.99" y1="-16.68" x2="20.32" y2="35.56" width="0" layer="19" extent="1-1"/>
+<wire x1="36.83" y1="13.97" x2="20.32" y2="35.56" width="0" layer="19" extent="1-1"/>
 </signal>
 <signal name="N$3">
+<contactref element="JP6" pad="1"/>
+<contactref element="JP11" pad="1"/>
+<contactref element="JP1" pad="1"/>
+<wire x1="17.78" y1="35.56" x2="17.78" y2="40.64" width="0" layer="19" extent="1-1"/>
+<wire x1="34.29" y1="13.97" x2="17.78" y2="35.56" width="0" layer="19" extent="1-1"/>
+</signal>
+<signal name="N$7">
 <contactref element="JP6" pad="3"/>
 <contactref element="JP11" pad="3"/>
-<contactref element="U$1" pad="5"/>
+<contactref element="JP1" pad="5"/>
 <wire x1="22.86" y1="35.56" x2="22.86" y2="40.64" width="0" layer="19" extent="1-1"/>
-<wire x1="18.53" y1="-16.68" x2="22.86" y2="35.56" width="0" layer="19" extent="1-1"/>
+<wire x1="39.37" y1="13.97" x2="22.86" y2="35.56" width="0" layer="19" extent="1-1"/>
 </signal>
-<signal name="3V3@1">
-<contactref element="JP6" pad="1"/>
-<contactref element="JP11" pad="1"/>
-<contactref element="U$1" pad="1"/>
-<wire x1="17.78" y1="35.56" x2="17.78" y2="40.64" width="0" layer="19" extent="1-1"/>
-<wire x1="13.45" y1="-16.68" x2="17.78" y2="35.56" width="0" layer="19" extent="1-1"/>
-</signal>
-<signal name="N$1">
-<contactref element="R1" pad="2"/>
-<contactref element="LED1" pad="A"/>
-<wire x1="39.37" y1="58.42" x2="30.48" y2="57.15" width="0" layer="19" extent="1-1"/>
+<signal name="N$6">
+<contactref element="DC-DC" pad="3"/>
+<contactref element="JP1" pad="2"/>
+<wire x1="5.08" y1="27.94" x2="34.29" y2="16.51" width="0" layer="19" extent="1-1"/>
 </signal>
 </signals>
