File: doc/pcb/OttoPi01/OttoPi01.brd (EAGLE design)
At the start: 53.3 x 64.4 mm, 20 parts

Commit message: update pcb
Parts:
- moved DC-DC 7.62 mm to (69.8, 72.4)
- moved C1 6.35 mm to (78.7, 27.9)
- moved SP 5.68 mm to (96.5, 27.9)
- moved VOL 5.68 mm to (96.5, 20.3), turned to 270 degrees
- moved AMPIN 5.08 mm to (81.3, 27.9)
- moved AMPOUT 5.08 mm to (88.9, 27.9)
- moved AUDIO 3.59 mm to (96.5, 24.1), turned to 90 degrees
- moved SV3 2.54 mm to (97.8, 41.9)
- moved RPI1 2.54 mm to (53.3, 48.3)
- moved RPI2 2.54 mm to (58.4, 48.3)
- moved SV1 2.54 mm to (97.8, 52.1)
- moved SV2 2.54 mm to (97.8, 47.0)
- moved SV4 2.54 mm to (97.8, 36.8)
- moved BAT 2.54 mm to (95.2, 77.5)
Connections:
- removed net N$40: RPI1.10, RPI2.10
- net GND: now also RPI1.10, RPI2.10
Routing:
- net GND: track 135.9 -> 188.8 mm
- net N$13: track 82.5 -> 95.2 mm
- net N$5: track 8.89 -> 16.5 mm
- net N$40: track 5.90 -> 0.00 mm
- net N$7: track 7.62 -> 10.2 mm
- net N$4: track 5.08 -> 7.62 mm
- net N$12: track 5.08 -> 7.62 mm
- net N$8: track 30.5 -> 27.9 mm
- net N$22: track 6.13 -> 6.88 mm
Other:
- board size 53.3 x 64.4 mm -> 55.9 x 64.4 mm
