File: doc/pcb/OttoPi01/OttoPi01.sch (EAGLE design)
At the start: 16 parts

Commit message: pcb
Parts:
- added JP1: (no value), pinhead:PINHD-2X20
Connections:
- removed net 3V3@1: JP11.1, JP6.1, U$1.3V3@1
- removed net 5V0@1: DC-DC.3, U$1.5V0@1
- removed net GND@8: U$1.GND@8
- new net N$4: AMP.2, C1.2
- new net N$5: AMP.3, C1.1
- new net N$6: DC-DC.3, JP1.2
- new net N$7: JP1.5, JP11.3, JP6.3
- net GND: now also JP1.6
- net N$2: now also JP1.3; no longer U$1.GPIO2/SDA1
- net N$3: now also JP1.1, JP11.1, JP6.1; no longer JP11.3, JP6.3, U$1.GPIO3/SCL1
Other:
- moved on the sheet: C1, JP11, JP6, U$1
Changed lines of the file:
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@@
 <part name="GND5" library="supply1" library_urn="urn:adsk.eagle:library:371" deviceset="GND" device=""/>
 <part name="GND6" library="supply1" library_urn="urn:adsk.eagle:library:371" deviceset="GND" device=""/>
+<part name="JP1" library="pinhead" library_urn="urn:adsk.eagle:library:325" deviceset="PINHD-2X20" device="" package3d_urn="urn:adsk.eagle:package:22443/2"/>
 </parts>
 <sheets>
@@
 </plain>
 <instances>
-<instance part="U$1" gate="G$1" x="38.1" y="60.96" smashed="yes">
-<attribute name="NAME" x="17.78" y="96.52" size="1.27" layer="95" font="vector"/>
-<attribute name="VALUE" x="17.78" y="94.615" size="1.27" layer="96" font="vector"/>
+<instance part="U$1" gate="G$1" x="43.18" y="15.24" smashed="yes">
+<attribute name="NAME" x="22.86" y="50.8" size="1.27" layer="95" font="vector"/>
+<attribute name="VALUE" x="22.86" y="48.895" size="1.27" layer="96" font="vector"/>
 </instance>
 <instance part="LED1" gate="G$1" x="137.16" y="116.84" smashed="yes">
@@
 <attribute name="VALUE" x="182.88" y="52.07" size="1.778" layer="96" rot="R270"/>
 </instance>
-<instance part="JP6" gate="A" x="-12.7" y="93.98" smashed="yes" rot="R270">
-<attribute name="NAME" x="-4.445" y="100.33" size="1.778" layer="95" rot="R270"/>
-<attribute name="VALUE" x="-20.32" y="100.33" size="1.778" layer="96" rot="R270"/>
+<instance part="JP6" gate="A" x="-2.54" y="99.06" smashed="yes">
+<attribute name="NAME" x="-8.89" y="107.315" size="1.778" layer="95"/>
+<attribute name="VALUE" x="-8.89" y="91.44" size="1.778" layer="96"/>
 </instance>
 <instance part="DC-DC" gate="A" x="88.9" y="93.98" smashed="yes" rot="R270">
@@
 <attribute name="VALUE" x="66.04" y="104.14" size="1.778" layer="96"/>
 </instance>
-<instance part="GND3" gate="1" x="71.12" y="83.82" smashed="yes">
-<attribute name="VALUE" x="68.58" y="81.28" size="1.778" layer="96"/>
+<instance part="GND3" gate="1" x="78.74" y="76.2" smashed="yes">
+<attribute name="VALUE" x="76.2" y="73.66" size="1.778" layer="96"/>
 </instance>
 <instance part="GND4" gate="1" x="127" y="68.58" smashed="yes">
@@
 <attribute name="VALUE" x="118.11" y="118.618" size="1.778" layer="96"/>
 </instance>
-<instance part="C1" gate="G$1" x="149.86" y="60.96" smashed="yes">
-<attribute name="NAME" x="151.384" y="61.341" size="1.778" layer="95"/>
-<attribute name="VALUE" x="151.384" y="56.261" size="1.778" layer="96"/>
-</instance>
-<instance part="JP11" gate="A" x="-12.7" y="81.28" smashed="yes" rot="R270">
-<attribute name="NAME" x="-4.445" y="87.63" size="1.778" layer="95" rot="R270"/>
-<attribute name="VALUE" x="-20.32" y="87.63" size="1.778" layer="96" rot="R270"/>
-</instance>
-<instance part="GND5" gate="1" x="-17.78" y="60.96" smashed="yes">
-<attribute name="VALUE" x="-20.32" y="58.42" size="1.778" layer="96"/>
+<instance part="C1" gate="G$1" x="190.5" y="55.88" smashed="yes" rot="R90">
+<attribute name="NAME" x="190.119" y="57.404" size="1.778" layer="95" rot="R90"/>
+<attribute name="VALUE" x="195.199" y="57.404" size="1.778" layer="96" rot="R90"/>
+</instance>
+<instance part="JP11" gate="A" x="12.7" y="99.06" smashed="yes">
+<attribute name="NAME" x="6.35" y="107.315" size="1.778" layer="95"/>
+<attribute name="VALUE" x="6.35" y="91.44" size="1.778" layer="96"/>
+</instance>
+<instance part="GND5" gate="1" x="2.54" y="83.82" smashed="yes">
+<attribute name="VALUE" x="0" y="81.28" size="1.778" layer="96"/>
 </instance>
 <instance part="GND6" gate="1" x="137.16" y="109.22" smashed="yes">
 <attribute name="VALUE" x="134.62" y="106.68" size="1.778" layer="96"/>
+</instance>
+<instance part="JP1" gate="A" x="43.18" y="81.28" smashed="yes">
+<attribute name="NAME" x="36.83" y="107.315" size="1.778" layer="95"/>
+<attribute name="VALUE" x="36.83" y="50.8" size="1.778" layer="96"/>
 </instance>
 </instances>
@@
 </segment>
 <segment>
+<pinref part="LED1" gate="G$1" pin="C"/>
+<pinref part="GND6" gate="1" pin="GND"/>
+</segment>
+<segment>
+<pinref part="GND3" gate="1" pin="GND"/>
+<pinref part="JP1" gate="A" pin="6"/>
+<wire x1="48.26" y1="99.06" x2="78.74" y2="99.06" width="0.1524" layer="91"/>
+<wire x1="78.74" y1="99.06" x2="78.74" y2="78.74" width="0.1524" layer="91"/>
+</segment>
+<segment>
 <pinref part="JP11" gate="A" pin="4"/>
 <pinref part="JP6" gate="A" pin="4"/>
-<wire x1="-15.24" y1="96.52" x2="-15.24" y2="83.82" width="0.1524" layer="91"/>
-<wire x1="-15.24" y1="83.82" x2="-15.24" y2="68.58" width="0.1524" layer="91"/>
-<junction x="-15.24" y="83.82"/>
-<wire x1="-15.24" y1="68.58" x2="-17.78" y2="68.58" width="0.1524" layer="91"/>
+<wire x1="-5.08" y1="96.52" x2="2.54" y2="96.52" width="0.1524" layer="91"/>
 <pinref part="GND5" gate="1" pin="GND"/>
-<wire x1="-17.78" y1="68.58" x2="-17.78" y2="63.5" width="0.1524" layer="91"/>
-</segment>
-<segment>
-<pinref part="LED1" gate="G$1" pin="C"/>
-<pinref part="GND6" gate="1" pin="GND"/>
-</segment>
-</net>
-<net name="5V0@1" class="0">
-<segment>
-<pinref part="DC-DC" gate="A" pin="3"/>
-<wire x1="86.36" y1="96.52" x2="71.12" y2="96.52" width="0.1524" layer="91"/>
-<wire x1="71.12" y1="96.52" x2="71.12" y2="91.44" width="0.1524" layer="91"/>
-<pinref part="U$1" gate="G$1" pin="5V0@1"/>
-<wire x1="71.12" y1="91.44" x2="63.5" y2="91.44" width="0.1524" layer="91"/>
-</segment>
-</net>
-<net name="GND@8" class="0">
-<segment>
-<pinref part="U$1" gate="G$1" pin="GND@8"/>
-<pinref part="GND3" gate="1" pin="GND"/>
-<wire x1="63.5" y1="86.36" x2="71.12" y2="86.36" width="0.1524" layer="91"/>
+<wire x1="2.54" y1="96.52" x2="10.16" y2="96.52" width="0.1524" layer="91"/>
+<wire x1="2.54" y1="86.36" x2="2.54" y2="96.52" width="0.1524" layer="91"/>
+<junction x="2.54" y="96.52"/>
 </segment>
 </net>
@@
 <pinref part="SV1" gate="A" pin="4"/>
 <wire x1="104.14" y1="81.28" x2="109.22" y2="81.28" width="0.1524" layer="91"/>
+<wire x1="114.3" y1="83.82" x2="109.22" y2="83.82" width="0.1524" layer="91"/>
 </segment>
 </net>
@@
 </segment>
 </net>
-<net name="N$2" class="0">
-<segment>
-<pinref part="JP6" gate="A" pin="2"/>
-<pinref part="JP11" gate="A" pin="2"/>
-<wire x1="-10.16" y1="96.52" x2="-10.16" y2="83.82" width="0.1524" layer="91"/>
-<pinref part="U$1" gate="G$1" pin="GPIO2/SDA1"/>
-<wire x1="15.24" y1="88.9" x2="2.54" y2="88.9" width="0.1524" layer="91"/>
-<wire x1="2.54" y1="88.9" x2="2.54" y2="71.12" width="0.1524" layer="91"/>
-<wire x1="2.54" y1="71.12" x2="-10.16" y2="71.12" width="0.1524" layer="91"/>
-<wire x1="-10.16" y1="71.12" x2="-10.16" y2="83.82" width="0.1524" layer="91"/>
-<junction x="-10.16" y="83.82"/>
-</segment>
-</net>
-<net name="N$3" class="0">
-<segment>
-<pinref part="JP6" gate="A" pin="3"/>
-<pinref part="JP11" gate="A" pin="3"/>
-<wire x1="-12.7" y1="96.52" x2="-12.7" y2="83.82" width="0.1524" layer="91"/>
-<pinref part="U$1" gate="G$1" pin="GPIO3/SCL1"/>
-<wire x1="15.24" y1="86.36" x2="5.08" y2="86.36" width="0.1524" layer="91"/>
-<wire x1="5.08" y1="86.36" x2="5.08" y2="68.58" width="0.1524" layer="91"/>
-<wire x1="5.08" y1="68.58" x2="-12.7" y2="68.58" width="0.1524" layer="91"/>
-<wire x1="-12.7" y1="68.58" x2="-12.7" y2="83.82" width="0.1524" layer="91"/>
-<junction x="-12.7" y="83.82"/>
-</segment>
-</net>
-<net name="3V3@1" class="0">
-<segment>
-<pinref part="JP6" gate="A" pin="1"/>
-<pinref part="JP11" gate="A" pin="1"/>
-<wire x1="-7.62" y1="96.52" x2="-7.62" y2="83.82" width="0.1524" layer="91"/>
-<wire x1="-7.62" y1="83.82" x2="-7.62" y2="73.66" width="0.1524" layer="91"/>
-<junction x="-7.62" y="83.82"/>
-<wire x1="-7.62" y1="73.66" x2="0" y2="73.66" width="0.1524" layer="91"/>
-<wire x1="0" y1="73.66" x2="0" y2="91.44" width="0.1524" layer="91"/>
-<pinref part="U$1" gate="G$1" pin="3V3@1"/>
-<wire x1="0" y1="91.44" x2="15.24" y2="91.44" width="0.1524" layer="91"/>
-</segment>
-</net>
 <net name="N$1" class="0">
 <segment>
@@
 </segment>
 </net>
+<net name="N$4" class="0">
+<segment>
+<pinref part="AMP" gate="A" pin="2"/>
+<wire x1="193.04" y1="48.26" x2="193.04" y2="53.34" width="0.1524" layer="91"/>
+<wire x1="193.04" y1="53.34" x2="195.58" y2="53.34" width="0.1524" layer="91"/>
+<pinref part="C1" gate="G$1" pin="2"/>
+<wire x1="195.58" y1="53.34" x2="195.58" y2="55.88" width="0.1524" layer="91"/>
+</segment>
+</net>
+<net name="N$5" class="0">
+<segment>
+<pinref part="AMP" gate="A" pin="3"/>
+<wire x1="190.5" y1="48.26" x2="190.5" y2="53.34" width="0.1524" layer="91"/>
+<wire x1="190.5" y1="53.34" x2="187.96" y2="53.34" width="0.1524" layer="91"/>
+<pinref part="C1" gate="G$1" pin="1"/>
+<wire x1="187.96" y1="53.34" x2="187.96" y2="55.88" width="0.1524" layer="91"/>
+</segment>
+</net>
+<net name="N$2" class="0">
+<segment>
+<pinref part="JP11" gate="A" pin="2"/>
+<junction x="10.16" y="101.6"/>
+<pinref part="JP1" gate="A" pin="3"/>
+<wire x1="40.64" y1="101.6" x2="10.16" y2="101.6" width="0.1524" layer="91"/>
+<pinref part="JP6" gate="A" pin="2"/>
+<wire x1="-5.08" y1="101.6" x2="10.16" y2="101.6" width="0.1524" layer="91"/>
+</segment>
+</net>
+<net name="N$3" class="0">
+<segment>
+<pinref part="JP11" gate="A" pin="1"/>
+<junction x="10.16" y="104.14"/>
+<pinref part="JP1" gate="A" pin="1"/>
+<wire x1="40.64" y1="104.14" x2="10.16" y2="104.14" width="0.1524" layer="91"/>
+<pinref part="JP6" gate="A" pin="1"/>
+<wire x1="-5.08" y1="104.14" x2="10.16" y2="104.14" width="0.1524" layer="91"/>
+</segment>
+</net>
+<net name="N$7" class="0">
+<segment>
+<pinref part="JP11" gate="A" pin="3"/>
+<junction x="10.16" y="99.06"/>
+<pinref part="JP1" gate="A" pin="5"/>
+<wire x1="40.64" y1="99.06" x2="10.16" y2="99.06" width="0.1524" layer="91"/>
+<pinref part="JP6" gate="A" pin="3"/>
+<wire x1="-5.08" y1="99.06" x2="10.16" y2="99.06" width="0.1524" layer="91"/>
+</segment>
+</net>
+<net name="N$6" class="0">
+<segment>
+<pinref part="DC-DC" gate="A" pin="3"/>
+<pinref part="JP1" gate="A" pin="2"/>
+<wire x1="48.26" y1="104.14" x2="86.36" y2="104.14" width="0.1524" layer="91"/>
+<wire x1="86.36" y1="104.14" x2="86.36" y2="96.52" width="0.1524" layer="91"/>
+</segment>
+</net>
