File: pcb/OttoPi02/OttoPi02.sch (EAGLE design)
At the start: 22 parts

Commit message: update pcb
Parts:
- added 5V_A, BAT_B, GND_A, GND_B: (no value), wirepad:1,6/0,9
- renumbered AUDIO to AIN, S2 to SW
Connections:
- removed net N$18: RPI1.5, RPI2.5
- net GND: now also GND_A.P, GND_B.P, RPI1.5, RPI2.5
- net N$13: now also BAT_B.P
- net N$5: now also 5V_A.P
Changed lines of the file:
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@@
 <part name="I2CIN" library="pinhead" library_urn="urn:adsk.eagle:library:325" deviceset="PINHD-1X3" device="" package3d_urn="urn:adsk.eagle:package:22458/2"/>
 <part name="DC-DC" library="pinhead" library_urn="urn:adsk.eagle:library:325" deviceset="PINHD-1X3" device="" package3d_urn="urn:adsk.eagle:package:22458/2"/>
-<part name="S2" library="switch" library_urn="urn:adsk.eagle:library:380" deviceset="TL36PO" device="" package3d_urn="urn:adsk.eagle:package:27745/1"/>
+<part name="SW" library="switch" library_urn="urn:adsk.eagle:library:380" deviceset="TL36PO" device="" package3d_urn="urn:adsk.eagle:package:27745/1"/>
 <part name="BAT" library="pinhead" library_urn="urn:adsk.eagle:library:325" deviceset="PINHD-1X2" device="" package3d_urn="urn:adsk.eagle:package:22435/2"/>
 <part name="5V" library="pinhead" library_urn="urn:adsk.eagle:library:325" deviceset="PINHD-1X2" device="" package3d_urn="urn:adsk.eagle:package:22435/2"/>
@@
 <part name="GND6" library="supply1" library_urn="urn:adsk.eagle:library:371" deviceset="GND" device=""/>
 <part name="C1" library="rcl" library_urn="urn:adsk.eagle:library:334" deviceset="C-EU" device="025-024X044" package3d_urn="urn:adsk.eagle:package:23630/1"/>
-<part name="AUDIO" library="pinhead" library_urn="urn:adsk.eagle:library:325" deviceset="PINHD-1X1" device="" package3d_urn="urn:adsk.eagle:package:22485/2"/>
+<part name="AIN" library="pinhead" library_urn="urn:adsk.eagle:library:325" deviceset="PINHD-1X1" device="" package3d_urn="urn:adsk.eagle:package:22485/2"/>
 <part name="LED1" library="led" library_urn="urn:adsk.eagle:library:259" deviceset="LED" device="3MM" package3d_urn="urn:adsk.eagle:package:15797/1"/>
 <part name="GND4" library="supply1" library_urn="urn:adsk.eagle:library:371" deviceset="GND" device=""/>
@@
 <part name="I2C1" library="pinhead" library_urn="urn:adsk.eagle:library:325" deviceset="PINHD-1X4" device="" package3d_urn="urn:adsk.eagle:package:22407/2"/>
 <part name="SV5" library="pinhead" library_urn="urn:adsk.eagle:library:325" deviceset="PINHD-1X4" device="" package3d_urn="urn:adsk.eagle:package:22407/2"/>
+<part name="GND_A" library="wirepad" library_urn="urn:adsk.eagle:library:412" deviceset="1,6/0,9" device="" package3d_urn="urn:adsk.eagle:package:30840/1"/>
+<part name="5V_A" library="wirepad" library_urn="urn:adsk.eagle:library:412" deviceset="1,6/0,9" device="" package3d_urn="urn:adsk.eagle:package:30840/1"/>
+<part name="BAT_B" library="wirepad" library_urn="urn:adsk.eagle:library:412" deviceset="1,6/0,9" device="" package3d_urn="urn:adsk.eagle:package:30840/1"/>
+<part name="GND_B" library="wirepad" library_urn="urn:adsk.eagle:library:412" deviceset="1,6/0,9" device="" package3d_urn="urn:adsk.eagle:package:30840/1"/>
 </parts>
 <sheets>
@@
 <attribute name="VALUE" x="99.06" y="62.23" size="1.778" layer="96" rot="R270"/>
 </instance>
-<instance part="S2" gate="BEF1" x="137.16" y="78.74" smashed="yes" rot="R270">
+<instance part="SW" gate="BEF1" x="137.16" y="78.74" smashed="yes" rot="R270">
 <attribute name="NAME" x="134.62" y="73.66" size="1.778" layer="95"/>
 <attribute name="VALUE" x="134.62" y="71.12" size="1.778" layer="96"/>
@@
 <attribute name="VALUE" x="92.456" y="40.259" size="1.778" layer="96" rot="R180"/>
 </instance>
-<instance part="AUDIO" gate="G$1" x="124.46" y="17.78" smashed="yes" rot="R270">
+<instance part="AIN" gate="G$1" x="124.46" y="17.78" smashed="yes" rot="R270">
 <attribute name="NAME" x="127.635" y="24.13" size="1.778" layer="95" rot="R270"/>
 <attribute name="VALUE" x="119.38" y="24.13" size="1.778" layer="96" rot="R270"/>
@@
 <attribute name="VALUE" x="109.22" y="-39.37" size="1.778" layer="96" rot="R270"/>
 </instance>
-<instance part="GND7" gate="1" x="152.4" y="-71.12" smashed="yes">
-<attribute name="VALUE" x="149.86" y="-73.66" size="1.778" layer="96"/>
+<instance part="GND7" gate="1" x="172.72" y="-109.22" smashed="yes">
+<attribute name="VALUE" x="170.18" y="-111.76" size="1.778" layer="96"/>
 </instance>
 <instance part="I2C1" gate="A" x="10.16" y="48.26" smashed="yes" rot="R270">
@@
 <attribute name="NAME" x="80.01" y="107.315" size="1.778" layer="95"/>
 <attribute name="VALUE" x="73.66" y="118.11" size="1.778" layer="96" rot="R270"/>
+</instance>
+<instance part="GND_A" gate="1" x="73.66" y="68.58" smashed="yes">
+<attribute name="NAME" x="72.517" y="70.4342" size="1.778" layer="95"/>
+<attribute name="VALUE" x="72.517" y="65.278" size="1.778" layer="96"/>
+</instance>
+<instance part="5V_A" gate="1" x="86.36" y="73.66" smashed="yes">
+<attribute name="NAME" x="85.217" y="75.5142" size="1.778" layer="95"/>
+<attribute name="VALUE" x="85.217" y="70.358" size="1.778" layer="96"/>
+</instance>
+<instance part="BAT_B" gate="1" x="121.92" y="86.36" smashed="yes">
+<attribute name="NAME" x="120.777" y="88.2142" size="1.778" layer="95"/>
+<attribute name="VALUE" x="120.777" y="83.058" size="1.778" layer="96"/>
+</instance>
+<instance part="GND_B" gate="1" x="154.94" y="88.9" smashed="yes">
+<attribute name="NAME" x="153.797" y="90.7542" size="1.778" layer="95"/>
+<attribute name="VALUE" x="153.797" y="85.598" size="1.778" layer="96"/>
 </instance>
 </instances>
@@
 <wire x1="106.68" y1="68.58" x2="91.44" y2="68.58" width="0.1524" layer="91"/>
 <junction x="91.44" y="68.58"/>
+<pinref part="GND_A" gate="1" pin="P"/>
+<wire x1="76.2" y1="68.58" x2="83.82" y2="68.58" width="0.1524" layer="91"/>
+<junction x="83.82" y="68.58"/>
 </segment>
 <segment>
@@
 <pinref part="GND3" gate="1" pin="GND"/>
 <wire x1="162.56" y1="81.28" x2="162.56" y2="73.66" width="0.1524" layer="91"/>
+<pinref part="GND_B" gate="1" pin="P"/>
+<wire x1="157.48" y1="88.9" x2="162.56" y2="88.9" width="0.1524" layer="91"/>
+<wire x1="162.56" y1="88.9" x2="162.56" y2="81.28" width="0.1524" layer="91"/>
+<junction x="162.56" y="81.28"/>
 </segment>
 <segment>
@@
 <wire x1="152.4" y1="-66.04" x2="152.4" y2="-50.8" width="0.1524" layer="91"/>
 <pinref part="GND7" gate="1" pin="GND"/>
-<wire x1="152.4" y1="-68.58" x2="152.4" y2="-66.04" width="0.1524" layer="91"/>
+<wire x1="172.72" y1="-106.68" x2="172.72" y2="-66.04" width="0.1524" layer="91"/>
+<wire x1="172.72" y1="-66.04" x2="152.4" y2="-66.04" width="0.1524" layer="91"/>
 <junction x="152.4" y="-66.04"/>
+<pinref part="RPI2" gate="A" pin="5"/>
+<wire x1="157.48" y1="-43.18" x2="157.48" y2="-33.02" width="0.1524" layer="91"/>
+<pinref part="RPI1" gate="A" pin="5"/>
+<wire x1="157.48" y1="-33.02" x2="93.98" y2="-33.02" width="0.1524" layer="91"/>
+<wire x1="93.98" y1="-33.02" x2="93.98" y2="-43.18" width="0.1524" layer="91"/>
+<wire x1="157.48" y1="-33.02" x2="172.72" y2="-33.02" width="0.1524" layer="91"/>
+<junction x="157.48" y="-33.02"/>
+<wire x1="172.72" y1="-33.02" x2="172.72" y2="-66.04" width="0.1524" layer="91"/>
+<junction x="172.72" y="-66.04"/>
 </segment>
 <segment>
@@
 <wire x1="104.14" y1="58.42" x2="104.14" y2="66.04" width="0.1524" layer="91"/>
 <wire x1="104.14" y1="66.04" x2="93.98" y2="66.04" width="0.1524" layer="91"/>
+<pinref part="5V_A" gate="1" pin="P"/>
+<wire x1="88.9" y1="73.66" x2="93.98" y2="73.66" width="0.1524" layer="91"/>
+<wire x1="93.98" y1="73.66" x2="93.98" y2="66.04" width="0.1524" layer="91"/>
+<junction x="93.98" y="66.04"/>
 </segment>
 </net>
@@
 <pinref part="BAT" gate="G$1" pin="2"/>
 <wire x1="149.86" y1="73.66" x2="149.86" y2="81.28" width="0.1524" layer="91"/>
-<pinref part="S2" gate="BEF1" pin="O"/>
+<pinref part="SW" gate="BEF1" pin="O"/>
 <wire x1="142.24" y1="81.28" x2="149.86" y2="81.28" width="0.1524" layer="91"/>
 </segment>
@@
 <wire x1="119.38" y1="48.26" x2="119.38" y2="78.74" width="0.1524" layer="91"/>
 <junction x="119.38" y="78.74"/>
-<pinref part="S2" gate="BEF1" pin="P"/>
+<pinref part="SW" gate="BEF1" pin="P"/>
 <pinref part="R1" gate="G$1" pin="2"/>
 <wire x1="127" y1="76.2" x2="127" y2="78.74" width="0.1524" layer="91"/>
@@
 <wire x1="83.82" y1="114.3" x2="83.82" y2="121.92" width="0.1524" layer="91"/>
 <junction x="83.82" y="121.92"/>
+<pinref part="BAT_B" gate="1" pin="P"/>
+<wire x1="124.46" y1="86.36" x2="127" y2="86.36" width="0.1524" layer="91"/>
+<wire x1="127" y1="86.36" x2="127" y2="78.74" width="0.1524" layer="91"/>
 </segment>
 </net>
@@
 <segment>
 <pinref part="VOL" gate="G$1" pin="1"/>
-<pinref part="AUDIO" gate="G$1" pin="1"/>
+<pinref part="AIN" gate="G$1" pin="1"/>
 <wire x1="111.76" y1="20.32" x2="111.76" y2="27.94" width="0.1524" layer="91"/>
 <wire x1="111.76" y1="27.94" x2="124.46" y2="27.94" width="0.1524" layer="91"/>
@@
 </segment>
 </net>
-<net name="N$18" class="0">
-<segment>
-<pinref part="RPI2" gate="A" pin="5"/>
-<wire x1="157.48" y1="-43.18" x2="157.48" y2="-33.02" width="0.1524" layer="91"/>
-<pinref part="RPI1" gate="A" pin="5"/>
-<wire x1="157.48" y1="-33.02" x2="93.98" y2="-33.02" width="0.1524" layer="91"/>
-<wire x1="93.98" y1="-33.02" x2="93.98" y2="-43.18" width="0.1524" layer="91"/>
-</segment>
-</net>
