File: pcb/OttoPi04/OttoPi04.brd (EAGLE design)
At the start: 48.3 x 63.5 mm, 26 parts

Commit message: pcb/OttoPi04
Parts:
- EXT: device pinhead:2X20 -> pinhead:2X20/90
- moved EXT 5.08 mm to (6.35, 34.3)
Connections:
- net N$30: no longer EXT.16
Routing:
- net GND: track 49.1 -> 0.74 mm
- net N$5: track 6.13 -> 5.39 mm
- net N$4: track 6.13 -> 5.39 mm
- net N$17: track 6.13 -> 5.39 mm
- net N$2: track 6.13 -> 5.39 mm
- net N$14: track 6.13 -> 5.39 mm
- net N$13: track 6.13 -> 5.39 mm
- net N$12: track 6.13 -> 5.39 mm
- net N$10: track 6.13 -> 5.39 mm
- net 3V: track 6.13 -> 5.39 mm
- net N$7: track 6.13 -> 5.39 mm
- net N$6: track 6.13 -> 5.39 mm
- net N$39: track 6.13 -> 5.39 mm
- net N$38: track 6.13 -> 5.39 mm
- net N$32: track 6.13 -> 5.39 mm
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