File: pcb/OttoPi04/OttoPi04.sch (EAGLE design)
At the start: 26 parts

Commit message: pcb/OttoPi04
Parts:
- EXT: device pinhead:PINHD-2X20 -> pinhead:PINHD-2X20/90
Connections:
- net N$30: no longer EXT.16
Other:
- moved on the sheet: AMPOUT, EXT, SP
