File: pcb/OttoPi04/OttoPi04.sch (EAGLE design)
At the start: 26 parts

Commit message: pcb
Parts:
- BAT: device pinhead:PINHD-1X2 -> adafruit:JST_2PIN-THM
- EXT: device pinhead:PINHD-2X20 -> con-lstb:MA20-2W
- RPI: device pinhead:PINHD-2X20 -> con-lsta:FE20-2
Connections:
- net 3V3 renamed +3V3
- net 5V renamed +5V
- removed net 3V: EXT.1, RPI.2
- removed net 4V: AMPIN.4, BAT_B.P, DC-DC.1, R1.2, SV1.2, SV2.2, SV3.2, SV4.2, SV5.2, SW.P
- removed net 5V1: EXT.2, RPI.1
- removed net 5V2: EXT.4, RPI.3
- removed net N$1: EXT.28, RPI.27
- removed net N$10: EXT.7, RPI.8
- removed net N$12: EXT.11, RPI.12
- removed net N$13: EXT.13, RPI.14
- removed net N$14: EXT.15, RPI.16
- removed net N$17: EXT.19, RPI.20
- removed net N$18: EXT.21, RPI.22
- removed net N$19: EXT.23, RPI.24
- removed net N$2: EXT.17, RPI.18
- removed net N$21: EXT.27, RPI.28
- removed net N$22: EXT.29, RPI.30
- removed net N$23: EXT.31, RPI.32
- removed net N$24: EXT.33, RPI.34
- removed net N$25: EXT.35, RPI.36
- removed net N$26: EXT.37, RPI.38
- removed net N$28: EXT.12, RPI.11
- removed net N$30: EXT.16, RPI.15
- removed net N$31: EXT.40, RPI.39
- removed net N$32: EXT.38, RPI.37
- removed net N$35: EXT.32, RPI.31
- removed net N$38: EXT.26, RPI.25
- removed net N$39: EXT.24, RPI.23
- removed net N$4: EXT.3, RPI.4
- removed net N$41: EXT.18, RPI.17
- removed net N$43: EXT.10, RPI.9
- removed net N$5: EXT.5, RPI.6
- removed net N$6: EXT.22, RPI.21
- removed net N$7: EXT.36, RPI.35
- removed net N$9: EXT.8, RPI.7
- new net +3V3-S1: EXT.1, RPI.1
- new net +3V3-S2: EXT.17, RPI.17
- new net +4V_S: BAT.2, SW.O
- new net +5V-S1: EXT.2, RPI.2
- new net +5V-S2: EXT.4, RPI.4
- new net GPIO0: EXT.27, RPI.27
- new net GPIO1: EXT.28, RPI.28
- new net GPIO10: EXT.19, RPI.19
- new net GPIO11: EXT.23, RPI.23
- new net GPIO12: EXT.32, RPI.32
- new net GPIO13: EXT.33, RPI.33
- new net GPIO14: EXT.8, RPI.8
- new net GPIO15: EXT.10, RPI.10
- new net GPIO16: EXT.36, RPI.36
- new net GPIO17: EXT.11, RPI.11
- new net GPIO18: EXT.12, RPI.12
- new net GPIO19: EXT.35, RPI.35
- new net GPIO20: EXT.38, RPI.38
- new net GPIO21: EXT.40, RPI.40
- new net GPIO22: EXT.15, RPI.15
- new net GPIO23: EXT.16, RPI.16
- new net GPIO24: EXT.18, RPI.18
- new net GPIO25: EXT.22, RPI.22
- new net GPIO26: EXT.37, RPI.37
- new net GPIO27: EXT.13, RPI.13
- new net GPIO4: EXT.7, RPI.7
- new net GPIO5: EXT.29, RPI.29
- new net GPIO6: EXT.31, RPI.31
- new net GPIO7: EXT.26, RPI.26
- new net GPIO8: EXT.24, RPI.24
- new net GPIO9: EXT.21, RPI.21
- new net SCL-S: EXT.5, RPI.5
- new net SDA-S: EXT.3, RPI.3
- net BAT+: now also AMPIN.4, BAT_B.P, DC-DC.1, R1.2, SV1.2, SV2.2, SV3.2, SV4.2, SV5.2, SW.P; no longer BAT.2, SW.O
- net GND: now also AMPIN.1, RPI.14, RPI.20, RPI.25, RPI.30, RPI.34, RPI.39, RPI.6, RPI.9; no longer RPI.10, RPI.13, RPI.19, RPI.26, RPI.29, RPI.33, RPI.40, RPI.5
Other:
- moved on the sheet: 5V, 5V_A, AIN, AMPIN, AMPOUT, BAT, BAT_B, C1, DC-DC, GND_A, GND_B, I2C1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

Commit message: pcb
Parts:
- removed SV5: (no value), pinhead:PINHD-1X4
- 5V_A: value (none) -> 5V
- GND_A: value (none) -> G
- renumbered GND_B to G
Connections:
- removed net SV5: SV5.3, SV5.4
- net BAT+: no longer SV5.2
- net GND: no longer SV5.1
Changed lines of the file:
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@@
 <part name="R1" library="rcl" library_urn="urn:adsk.eagle:library:334" deviceset="R-EU_" device="0204/7" package3d_urn="urn:adsk.eagle:package:23498/2"/>
 <part name="I2C1" library="pinhead" library_urn="urn:adsk.eagle:library:325" deviceset="PINHD-1X4" device="" package3d_urn="urn:adsk.eagle:package:22407/2"/>
-<part name="SV5" library="pinhead" library_urn="urn:adsk.eagle:library:325" deviceset="PINHD-1X4" device="" package3d_urn="urn:adsk.eagle:package:22407/2"/>
-<part name="GND_A" library="wirepad" library_urn="urn:adsk.eagle:library:412" deviceset="1,6/0,9" device="" package3d_urn="urn:adsk.eagle:package:30840/1"/>
-<part name="5V_A" library="wirepad" library_urn="urn:adsk.eagle:library:412" deviceset="1,6/0,9" device="" package3d_urn="urn:adsk.eagle:package:30840/1"/>
+<part name="GND_A" library="wirepad" library_urn="urn:adsk.eagle:library:412" deviceset="1,6/0,9" device="" package3d_urn="urn:adsk.eagle:package:30840/1" value="G"/>
+<part name="5V_A" library="wirepad" library_urn="urn:adsk.eagle:library:412" deviceset="1,6/0,9" device="" package3d_urn="urn:adsk.eagle:package:30840/1" value="5V"/>
 <part name="BAT_B" library="wirepad" library_urn="urn:adsk.eagle:library:412" deviceset="1,6/0,9" device="" package3d_urn="urn:adsk.eagle:package:30840/1"/>
-<part name="GND_B" library="wirepad" library_urn="urn:adsk.eagle:library:412" deviceset="1,6/0,9" device="" package3d_urn="urn:adsk.eagle:package:30840/1"/>
+<part name="G" library="wirepad" library_urn="urn:adsk.eagle:library:412" deviceset="1,6/0,9" device="" package3d_urn="urn:adsk.eagle:package:30840/1"/>
 <part name="RPI" library="con-lsta" library_urn="urn:adsk.eagle:library:161" deviceset="FE20-2" device="" package3d_urn="urn:adsk.eagle:package:8184/1"/>
 <part name="EXT" library="con-lstb" library_urn="urn:adsk.eagle:library:162" deviceset="MA20-2W" device="" package3d_urn="urn:adsk.eagle:package:8363/1"/>
@@
 <attribute name="VALUE" x="171.45" y="86.36" size="1.778" layer="96"/>
 </instance>
-<instance part="SV5" gate="A" x="233.68" y="134.62" smashed="yes">
-<attribute name="NAME" x="238.125" y="133.35" size="1.778" layer="95" rot="R90"/>
-<attribute name="VALUE" x="227.33" y="127" size="1.778" layer="96"/>
-</instance>
 <instance part="GND_A" gate="1" x="20.32" y="38.1" smashed="yes">
 <attribute name="NAME" x="16.637" y="39.9542" size="1.778" layer="95"/>
@@
 <attribute name="VALUE" x="16.637" y="116.078" size="1.778" layer="96"/>
 </instance>
-<instance part="GND_B" gate="1" x="58.42" y="114.3" smashed="yes" rot="R180">
+<instance part="G" gate="1" x="58.42" y="114.3" smashed="yes" rot="R180">
 <attribute name="NAME" x="64.643" y="117.5258" size="1.778" layer="95" rot="R180"/>
 <attribute name="VALUE" x="59.563" y="117.602" size="1.778" layer="96" rot="R180"/>
@@
 <attribute name="VALUE" x="165.1" y="58.42" size="1.778" layer="96" rot="R180"/>
 </instance>
-<instance part="P+6" gate="1" x="218.44" y="144.78" smashed="yes">
-<attribute name="VALUE" x="220.98" y="147.32" size="1.778" layer="96" rot="R180"/>
+<instance part="P+6" gate="1" x="218.44" y="129.54" smashed="yes">
+<attribute name="VALUE" x="220.98" y="132.08" size="1.778" layer="96" rot="R180"/>
 </instance>
 <instance part="P+7" gate="1" x="50.8" y="63.5" smashed="yes">
@@
 <wire x1="48.26" y1="109.22" x2="48.26" y2="114.3" width="0.1524" layer="91"/>
 <wire x1="53.34" y1="114.3" x2="48.26" y2="114.3" width="0.1524" layer="91"/>
-<pinref part="GND_B" gate="1" pin="P"/>
+<pinref part="G" gate="1" pin="P"/>
 <wire x1="55.88" y1="114.3" x2="53.34" y2="114.3" width="0.1524" layer="91"/>
 <junction x="53.34" y="114.3"/>
@@
 <wire x1="220.98" y1="121.92" x2="220.98" y2="104.14" width="0.1524" layer="91"/>
 <junction x="220.98" y="104.14"/>
-<pinref part="SV5" gate="A" pin="1"/>
-<wire x1="231.14" y1="139.7" x2="220.98" y2="139.7" width="0.1524" layer="91"/>
-<wire x1="220.98" y1="139.7" x2="220.98" y2="121.92" width="0.1524" layer="91"/>
-<junction x="220.98" y="121.92"/>
 <pinref part="GND5" gate="1" pin="GND"/>
 <wire x1="220.98" y1="55.88" x2="220.98" y2="68.58" width="0.1524" layer="91"/>
@@
 <net name="AIN2" class="0">
 <segment>
-<pinref part="AMPIN" gate="A" pin="2"/>
-<wire x1="157.48" y1="45.72" x2="162.56" y2="45.72" width="0.1524" layer="91"/>
-<pinref part="VOL" gate="G$1" pin="2"/>
-<wire x1="157.48" y1="33.02" x2="162.56" y2="33.02" width="0.1524" layer="91"/>
 <wire x1="162.56" y1="33.02" x2="162.56" y2="45.72" width="0.1524" layer="91"/>
 <pinref part="C1" gate="G$1" pin="2"/>
 <wire x1="165.1" y1="45.72" x2="162.56" y2="45.72" width="0.1524" layer="91"/>
+<pinref part="AMPIN" gate="A" pin="2"/>
+<wire x1="157.48" y1="45.72" x2="162.56" y2="45.72" width="0.1524" layer="91"/>
 <junction x="162.56" y="45.72"/>
+<pinref part="VOL" gate="G$1" pin="2"/>
+<wire x1="157.48" y1="33.02" x2="162.56" y2="33.02" width="0.1524" layer="91"/>
 </segment>
 </net>
@@
 <pinref part="LED1" gate="G$1" pin="A"/>
 <wire x1="25.4" y1="99.06" x2="25.4" y2="96.52" width="0.1524" layer="91"/>
-</segment>
-</net>
-<net name="SV5" class="0">
-<segment>
-<pinref part="SV5" gate="A" pin="4"/>
-<wire x1="231.14" y1="132.08" x2="226.06" y2="132.08" width="0.1524" layer="91"/>
-<wire x1="226.06" y1="132.08" x2="226.06" y2="134.62" width="0.1524" layer="91"/>
-<pinref part="SV5" gate="A" pin="3"/>
-<wire x1="226.06" y1="134.62" x2="231.14" y2="134.62" width="0.1524" layer="91"/>
 </segment>
 </net>
@@
 <junction x="218.44" y="101.6"/>
 <junction x="218.44" y="119.38"/>
-<wire x1="218.44" y1="137.16" x2="218.44" y2="119.38" width="0.1524" layer="91"/>
-<pinref part="SV5" gate="A" pin="2"/>
-<wire x1="231.14" y1="137.16" x2="218.44" y2="137.16" width="0.1524" layer="91"/>
+<wire x1="218.44" y1="127" x2="218.44" y2="119.38" width="0.1524" layer="91"/>
 <pinref part="P+6" gate="1" pin="V+"/>
-<wire x1="218.44" y1="142.24" x2="218.44" y2="137.16" width="0.1524" layer="91"/>
-<junction x="218.44" y="137.16"/>
-</segment>
-</net>
+</segment>
+</net>

Commit message: pcb
Parts:
- removed 5V_A: 5V, wirepad:1,6/0,9
- removed BAT_B, G: (no value), wirepad:1,6/0,9
- removed C1: (no value), rcl:C-EU025-024X044
- removed GND_A: G, wirepad:1,6/0,9
- removed I2C2: (no value), pinhead:PINHD-1X4
- R1: value (none) -> 1K
Connections:
- new net N$1: AMPOUT.1
- new net N$2: AMPOUT.2
- net +3V3: no longer I2C2.1
- net +5V: no longer 5V_A.P
- net AIN2: no longer C1.2
- net BAT+: now also SW.S; no longer BAT_B.P
- net GND: no longer C1.1, G.P, GND_A.P, I2C2.4
- net SCL: no longer I2C2.3
- net SDL: no longer I2C2.2
- net SP+: no longer AMPOUT.1
- net SP-: no longer AMPOUT.2
Other:
- moved on the sheet: AIN, AMPIN, AMPOUT, SP, VOL
