File: pcb/OttoPi05-RPi3BHAT/OttoPi05.brd (EAGLE design)
At the start: 65 x 55 mm, 18 parts

Commit message: update
Parts:
- added C1: (no value), rcl:C025-024X044
- moved I2CIN 19.3 mm to (20.3, 27.9)
- moved I2C1 19.3 mm to (19.1, 33.0)
- moved AIN 15.5 mm to (5.08, 35.6), turned to 180 degrees
- moved AMPOUT 10.5 mm to (5.08, 31.8), turned to 90 degrees
- moved R1 9.67 mm to (38.1, 41.9), turned to 270 degrees
- moved VOL 8.03 mm to (5.08, 39.4), turned to 90 degrees
- moved SV1 5.68 mm to (30.5, 44.5)
- moved SV2 5.68 mm to (25.4, 44.5)
- moved SV4 5.68 mm to (15.2, 44.5)
- moved P1 5.68 mm to (54.6, 48.3)
- moved SV3 5.68 mm to (20.3, 44.5)
- moved SW1 5.68 mm to (45.7, 48.3)
- moved LED1 5.08 mm to (36.8, 48.3)
- moved DCDC1 2.84 mm to (50.8, 26.7)
- moved AMP1 2.54 mm to (6.35, 21.6)
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Connections:
- net N$1 renamed +5V
- net N$4 renamed SP+
- net N$5 renamed SP-
- net N$7 renamed BAT+S
- removed net N$3: AMP1.IN+, VOL.2
- new net AIN: AMP1.IN+, C1.1, VOL.2
- new net GND14: EXT.14, RPI.14
- new net GND20: EXT.20, RPI.20
- new net GND25: EXT.25, RPI.25
- new net GND30: EXT.30, RPI.30
- new net GND34: EXT.34, RPI.34
- new net GND6: EXT.6, RPI.6
- new net GND9: EXT.9, RPI.9
- net BAT+: now also SW1.3
- net GND: now also C1.2; no longer EXT.14, EXT.20, EXT.25, EXT.30, EXT.34, EXT.6, EXT.9, RPI.14, RPI.20, RPI.25, RPI.30, RPI.34, RPI.6, RPI.9
Routing:
- net GND: track 0.00 -> 213.0 mm
- net BAT+: track 13.7 -> 61.1 mm
- net AIN: track 0.00 -> 40.6 mm
- net SP-: track 0.00 -> 12.7 mm
- net SP+: track 0.00 -> 7.62 mm
- net +5V-S1: track 0.00 -> 6.17 mm
- net SCL-S: track 0.00 -> 6.13 mm
- net GPIO7: track 0.00 -> 6.13 mm
- net GPIO4: track 0.00 -> 6.13 mm
- net GPIO18: track 0.00 -> 6.13 mm
- net GPIO17: track 0.00 -> 6.13 mm
- net GPIO15: track 0.00 -> 6.13 mm
- net GPIO14: track 0.00 -> 6.13 mm
- net GND6: track 0.00 -> 6.13 mm
- net GPIO19: track 0.00 -> 6.13 mm
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