File: pcb/OttoPi05-RPi3BHAT/OttoPi05.sch (EAGLE design)
At the start: 18 parts

Commit message: update
Parts:
- added C1: (no value), rcl:C-EU025-024X044
Connections:
- net N$1 renamed +5V
- net N$4 renamed SP+
- net N$5 renamed SP-
- net N$7 renamed BAT+S
- removed net N$3: AMP1.IN+, VOL.2
- new net AIN: AMP1.IN+, C1.1, VOL.2
- new net GND14: EXT.14, RPI.14
- new net GND20: EXT.20, RPI.20
- new net GND25: EXT.25, RPI.25
- new net GND30: EXT.30, RPI.30
- new net GND34: EXT.34, RPI.34
- new net GND6: EXT.6, RPI.6
- new net GND9: EXT.9, RPI.9
- net BAT+: now also SW1.3
- net GND: now also C1.2; no longer EXT.14, EXT.20, EXT.25, EXT.30, EXT.34, EXT.6, EXT.9, RPI.14, RPI.20, RPI.25, RPI.30, RPI.34, RPI.6, RPI.9
Other:
- moved on the sheet: AIN, AMP1, AMPOUT, P1, SW1, VOL
