File: pcb/OttoPi04-RPiZeroHAT/OttoPi04.sch (EAGLE design)
At the start: 19 parts

Commit message: pcb/OttoPi04-RPiZeroHAT
Parts:
- removed 5V, SP: (no value), pinhead:PINHD-1X2
- removed DC-DC: (no value), pinhead:PINHD-1X3
- added 5V1: (no value), pinhead:PINHD-1X2
- added DC/DC1: DC/DC-03_5V_480MA, ytani1:DC/DC-03_5V_480MA
Connections:
- removed net BAT+: AMPIN.4, DC-DC.1, R1.2, SV1.2, SV2.2, SV3.2, SV4.2, SW.P, SW.S
- removed net N$1: AMPOUT.1
- removed net N$2: AMPOUT.2
- removed net SP+: SP.1
- removed net SP-: SP.2
- new net V+: AMPIN.4, DC/DC1.VIN, R1.2, SV1.2, SV2.2, SV3.2, SV4.2, SW.P, SW.S
- net +5V: now also 5V1.2, DC/DC1.+5V; no longer 5V.1, DC-DC.3
- net GND: now also 5V1.1, DC/DC1.GND; no longer 5V.2, DC-DC.2
Other:
- moved on the sheet: AIN, AMPIN, AMPOUT, BAT, EXT, I2C1, I2CIN, LED1, R1, RPI, SV1, SV2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

Commit message: update
Connections:
- net V+: no longer SW.S
Changed lines of the file:
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@@
 <?xml version="1.0" encoding="utf-8"?>
 <!DOCTYPE eagle SYSTEM "eagle.dtd">
-<eagle version="9.6.0">
+<eagle version="9.6.2">
 <drawing>
 <settings>
@@
 <wire x1="53.34" y1="139.7" x2="53.34" y2="137.16" width="0.1524" layer="91"/>
 <wire x1="53.34" y1="134.62" x2="53.34" y2="137.16" width="0.1524" layer="91"/>
-<wire x1="55.88" y1="132.08" x2="55.88" y2="137.16" width="0.1524" layer="91"/>
-<junction x="55.88" y="137.16"/>
-<pinref part="SW" gate="BEF1" pin="S"/>
-<wire x1="66.04" y1="134.62" x2="68.58" y2="134.62" width="0.1524" layer="91"/>
-<wire x1="68.58" y1="134.62" x2="68.58" y2="132.08" width="0.1524" layer="91"/>
-<wire x1="55.88" y1="132.08" x2="68.58" y2="132.08" width="0.1524" layer="91"/>
 <pinref part="P+3" gate="1" pin="V+"/>
 <wire x1="53.34" y1="144.78" x2="53.34" y2="137.16" width="0.1524" layer="91"/>

Commit message: update
Parts:
- removed DC/DC1: DC/DC-03_5V_480MA, ytani1:DC/DC-03_5V_480MA
- added DCDC1: (no value), ytani1:DCDC-5V-0.48A
- BAT: device adafruit:JST_2PIN-THM -> ytani1:JST-PH2
- renumbered 5V1 to 5V
Connections:
- net +4V_S: now also BAT.1; no longer BAT.2
- net +5V: now also DCDC1.VOUT; no longer DC/DC1.+5V
- net GND: now also BAT.2, DCDC1.GND; no longer BAT.1, DC/DC1.GND
- net V+: now also DCDC1.VIN; no longer DC/DC1.VIN
Other:
- moved on the sheet: BAT
Changed lines of the file:
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@@
 <setting verticaltext="up"/>
 </settings>
-<grid distance="0.1" unitdist="inch" unit="inch" style="lines" multiple="1" display="no" altdistance="0.01" altunitdist="inch" altunit="inch"/>
+<grid distance="1.27" unitdist="mm" unit="mm" style="lines" multiple="2" display="yes" altdistance="0.01" altunitdist="inch" altunit="inch"/>
 <layers>
 <layer number="1" name="Top" color="4" fill="1" visible="no" active="no"/>
@@
 <part name="I2C1" library="pinhead" library_urn="urn:adsk.eagle:library:325" deviceset="PINHD-1X4" device="" package3d_urn="urn:adsk.eagle:package:22407/2"/>
 <part name="RPI" library="con-lsta" library_urn="urn:adsk.eagle:library:161" deviceset="FE20-2" device="" package3d_urn="urn:adsk.eagle:package:8184/1"/>
-<part name="EXT" library="con-lstb" library_urn="urn:adsk.eagle:library:162" deviceset="MA20-2W" device="" package3d_urn="urn:adsk.eagle:package:8363/1"/>
+<part name="EXT" library="con-lstb" deviceset="MA20-2W" device="" package3d_urn="urn:adsk.eagle:package:8363/1"/>
 <part name="+3V3" library="supply1" library_urn="urn:adsk.eagle:library:371" deviceset="+3V3" device=""/>
 <part name="+3V4" library="supply1" library_urn="urn:adsk.eagle:library:371" deviceset="+3V3" device=""/>
@@
 <part name="GND23" library="supply1" library_urn="urn:adsk.eagle:library:371" deviceset="GND" device=""/>
 <part name="+3V5" library="supply1" library_urn="urn:adsk.eagle:library:371" deviceset="+3V3" device=""/>
-<part name="BAT" library="adafruit" deviceset="JST_2PIN" device="-THM"/>
 <part name="FRAME1" library="frames" library_urn="urn:adsk.eagle:library:229" deviceset="A4L-LOC" device=""/>
-<part name="5V1" library="pinhead" library_urn="urn:adsk.eagle:library:325" deviceset="PINHD-1X2" device="" package3d_urn="urn:adsk.eagle:package:22435/2"/>
-<part name="DC/DC1" library="ytani1" deviceset="DC/DC-03_5V_480MA" device=""/>
+<part name="5V" library="pinhead" library_urn="urn:adsk.eagle:library:325" deviceset="PINHD-1X2" device="" package3d_urn="urn:adsk.eagle:package:22435/2"/>
 <part name="P+3" library="supply1" library_urn="urn:adsk.eagle:library:371" deviceset="V+" device="" value="BAT+"/>
+<part name="BAT" library="ytani1" deviceset="JST-PH2" device=""/>
+<part name="DCDC1" library="ytani1" deviceset="DCDC-5V-0.48A" device=""/>
 </parts>
 <sheets>
@@
 <attribute name="VALUE" x="33.02" y="111.76" size="1.778" layer="96"/>
 </instance>
-<instance part="GND3" gate="1" x="81.28" y="124.46" smashed="yes">
-<attribute name="VALUE" x="78.74" y="121.92" size="1.778" layer="96"/>
+<instance part="GND3" gate="1" x="73.66" y="132.08" smashed="yes">
+<attribute name="VALUE" x="71.12" y="129.54" size="1.778" layer="96"/>
 </instance>
 <instance part="GND5" gate="1" x="208.28" y="73.66" smashed="yes">
@@
 <attribute name="VALUE" x="119.38" y="147.32" size="1.778" layer="96" rot="R180"/>
 </instance>
-<instance part="BAT" gate="G$1" x="73.66" y="132.08" smashed="yes" rot="R270">
-<attribute name="NAME" x="72.39" y="127.635" size="1.778" layer="95"/>
-<attribute name="VALUE" x="68.58" y="138.43" size="1.778" layer="96" rot="R270"/>
-</instance>
 <instance part="FRAME1" gate="G$1" x="-2.54" y="-15.24" smashed="yes">
 <attribute name="DRAWING_NAME" x="214.63" y="0" size="2.54" layer="94"/>
@@
 <attribute name="SHEET" x="227.965" y="-10.16" size="2.54" layer="94"/>
 </instance>
-<instance part="5V1" gate="G$1" x="22.86" y="124.46" smashed="yes" rot="R180">
+<instance part="5V" gate="G$1" x="22.86" y="124.46" smashed="yes" rot="R180">
 <attribute name="NAME" x="18.415" y="125.73" size="1.778" layer="95" rot="R270"/>
 <attribute name="VALUE" x="29.21" y="129.54" size="1.778" layer="96" rot="R180"/>
 </instance>
-<instance part="DC/DC1" gate="G$1" x="25.4" y="134.62" smashed="yes">
-<attribute name="NAME" x="17.78" y="143.16" size="1.778" layer="95"/>
-<attribute name="VALUE" x="17.78" y="140.66" size="1.778" layer="96"/>
-</instance>
 <instance part="P+3" gate="1" x="53.34" y="147.32" smashed="yes">
 <attribute name="VALUE" x="55.88" y="149.86" size="1.778" layer="96" rot="R180"/>
+</instance>
+<instance part="BAT" gate="G$1" x="81.28" y="139.7" smashed="yes">
+<attribute name="NAME" x="76.2" y="143.002" size="1.778" layer="95"/>
+<attribute name="VALUE" x="76.2" y="132.334" size="1.778" layer="96"/>
+</instance>
+<instance part="DCDC1" gate="G$1" x="33.02" y="149.86" smashed="yes">
+<attribute name="NAME" x="27.94" y="153.67" size="1.778" layer="95"/>
 </instance>
 </instances>
@@
 <label x="15.24" y="7.62" size="1.778" layer="95"/>
 <pinref part="GND23" gate="1" pin="GND"/>
-</segment>
-<segment>
-<pinref part="GND3" gate="1" pin="GND"/>
-<wire x1="81.28" y1="127" x2="81.28" y2="139.7" width="0.1524" layer="91"/>
-<pinref part="BAT" gate="G$1" pin="1"/>
-<wire x1="76.2" y1="134.62" x2="76.2" y2="139.7" width="0.1524" layer="91"/>
-<wire x1="81.28" y1="139.7" x2="76.2" y2="139.7" width="0.1524" layer="91"/>
 </segment>
 <segment>
@@
 </segment>
 <segment>
-<pinref part="5V1" gate="G$1" pin="1"/>
+<pinref part="5V" gate="G$1" pin="1"/>
 <wire x1="25.4" y1="121.92" x2="35.56" y2="121.92" width="0.1524" layer="91"/>
 <wire x1="35.56" y1="121.92" x2="35.56" y2="134.62" width="0.1524" layer="91"/>
@@
 <wire x1="35.56" y1="116.84" x2="35.56" y2="121.92" width="0.1524" layer="91"/>
 <junction x="35.56" y="121.92"/>
-<pinref part="DC/DC1" gate="G$1" pin="GND"/>
-<wire x1="30.48" y1="134.62" x2="35.56" y2="134.62" width="0.1524" layer="91"/>
+<pinref part="DCDC1" gate="G$1" pin="GND"/>
+<wire x1="33.02" y1="134.62" x2="35.56" y2="134.62" width="0.1524" layer="91"/>
+<wire x1="33.02" y1="144.78" x2="33.02" y2="134.62" width="0.1524" layer="91"/>
+</segment>
+<segment>
+<pinref part="BAT" gate="G$1" pin="2"/>
+<wire x1="78.74" y1="137.16" x2="73.66" y2="137.16" width="0.1524" layer="91"/>
+<pinref part="GND3" gate="1" pin="GND"/>
+<wire x1="73.66" y1="137.16" x2="73.66" y2="134.62" width="0.1524" layer="91"/>
 </segment>
 </net>
@@
 <pinref part="P+4" gate="1" pin="V+"/>
 <wire x1="73.66" y1="144.78" x2="73.66" y2="139.7" width="0.1524" layer="91"/>
-<pinref part="BAT" gate="G$1" pin="2"/>
-<wire x1="73.66" y1="134.62" x2="73.66" y2="139.7" width="0.1524" layer="91"/>
+<pinref part="BAT" gate="G$1" pin="1"/>
+<wire x1="78.74" y1="139.7" x2="73.66" y2="139.7" width="0.1524" layer="91"/>
 <junction x="73.66" y="139.7"/>
 </segment>
@@
 <net name="+5V" class="0">
 <segment>
-<wire x1="33.02" y1="132.08" x2="33.02" y2="124.46" width="0.1524" layer="91"/>
-<pinref part="5V1" gate="G$1" pin="2"/>
-<wire x1="33.02" y1="124.46" x2="25.4" y2="124.46" width="0.1524" layer="91"/>
-<pinref part="DC/DC1" gate="G$1" pin="+5V"/>
-<wire x1="30.48" y1="132.08" x2="33.02" y2="132.08" width="0.1524" layer="91"/>
+<pinref part="5V" gate="G$1" pin="2"/>
+<pinref part="DCDC1" gate="G$1" pin="VOUT"/>
+<wire x1="40.64" y1="149.86" x2="43.18" y2="149.86" width="0.1524" layer="91"/>
+<wire x1="43.18" y1="149.86" x2="43.18" y2="124.46" width="0.1524" layer="91"/>
+<wire x1="43.18" y1="124.46" x2="25.4" y2="124.46" width="0.1524" layer="91"/>
 </segment>
 </net>
@@
 <pinref part="P+3" gate="1" pin="V+"/>
 <wire x1="53.34" y1="144.78" x2="53.34" y2="137.16" width="0.1524" layer="91"/>
-<pinref part="DC/DC1" gate="G$1" pin="VIN"/>
-<wire x1="30.48" y1="137.16" x2="53.34" y2="137.16" width="0.1524" layer="91"/>
-</segment>
-<segment>
+<wire x1="30.48" y1="137.16" x2="31.75" y2="137.16" width="0.1524" layer="91"/>
+<pinref part="DCDC1" gate="G$1" pin="VIN"/>
+<wire x1="31.75" y1="137.16" x2="53.34" y2="137.16" width="0.1524" layer="91"/>
+<wire x1="25.4" y1="149.86" x2="22.86" y2="149.86" width="0.1524" layer="91"/>
+<wire x1="22.86" y1="149.86" x2="22.86" y2="137.16" width="0.1524" layer="91"/>
+<wire x1="22.86" y1="137.16" x2="30.48" y2="137.16" width="0.1524" layer="91"/>
+</segment>
+<segment>
