File: pcb/OttoPi05a-RPi3BHAT/OttoPi05.brd (EAGLE design)
At the start: 65 x 55 mm, 26 parts

Commit message: update
Parts:
- AMP: device ytani1:PAM8012MOD -> ytani1:PAM8012MOD-A
Connections:
- net SP+: no longer AMP.SP+@2
- net SP-: no longer AMP.SP-@2
Routing:
- net BAT+S: track 5.35 -> 9.25 mm
Changed lines of the file:
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@@
 <attribute name="URL_AMAZON" value="https://www.amazon.co.jp/gp/product/B01LYVYQNO/" x="45.72" y="48.26" size="1.778" layer="27" rot="R180" display="off"/>
 </element>
-<element name="AMP" library="ytani1" package="PAM8012MOD" value="PAM8012MOD" x="6.35" y="21.59" smashed="yes" rot="R90">
+<element name="AMP" library="ytani1" package="PAM8012MOD-A" value="PAM8012MOD" x="6.35" y="21.59" smashed="yes" rot="R90">
 <attribute name="CHIP1" value="PAM8012" x="6.35" y="21.59" size="1.778" layer="27" rot="R90" display="off"/>
 <attribute name="NAME" x="0" y="15.24" size="1.016" layer="25"/>
@@
 <wire x1="17.78" y1="45.72" x2="22.86" y2="45.72" width="0.8128" layer="16"/>
 <wire x1="22.86" y1="45.72" x2="27.94" y2="45.72" width="0.8128" layer="16"/>
-<wire x1="43.18" y1="48.26" x2="45.72" y2="48.26" width="0.8128" layer="16"/>
-<wire x1="45.72" y1="48.26" x2="45.72" y2="43.18" width="0.8128" layer="16"/>
+<wire x1="39.37" y1="46.99" x2="41.91" y2="46.99" width="0.8128" layer="16"/>
+<wire x1="41.91" y1="46.99" x2="45.72" y2="43.18" width="0.8128" layer="16"/>
 <wire x1="45.72" y1="43.18" x2="57.8" y2="43.18" width="0.8128" layer="16"/>
 <wire x1="57.8" y1="39.92" x2="57.8" y2="43.18" width="0.8128" layer="16"/>
@@
 </signal>
 <signal name="SP+">
-<contactref element="AMP" pad="SP+@1"/>
-<contactref element="AMP" pad="SP+@2"/>
+<contactref element="AMP" pad="SP+@1" route="any" routetag="G$1.SP+"/>
 <wire x1="2.54" y1="25.4" x2="5.08" y2="25.4" width="0.8128" layer="16"/>
 <contactref element="SP" pad="1"/>
@@
 <signal name="SP-">
 <contactref element="AMP" pad="SP-@1"/>
-<contactref element="AMP" pad="SP-@2"/>
 <wire x1="7.62" y1="25.4" x2="10.16" y2="25.4" width="0.8128" layer="16"/>
 <wire x1="7.62" y1="33.02" x2="7.62" y2="25.4" width="0.6096" layer="16"/>
@@
 <contactref element="BAT" pad="1"/>
 <contactref element="PWR" pad="1"/>
-<wire x1="48.26" y1="48.26" x2="53.61" y2="48.26" width="0.8128" layer="16"/>
+<wire x1="44.45" y1="46.99" x2="53.61" y2="48.26" width="0.8128" layer="16"/>
 </signal>
 <signal name="GND14">
