File: pcb/OttoPi06a-RPi3AHAT/OttoPi06a-RPi3AHAT.brd (EAGLE design)
At the start: 56 x 65 mm, 28 parts

Commit message: pcb
Parts:
- moved VOL 1.80 mm to (1.27, 7.62)
- moved SP+ 1.80 mm to (1.27, 2.54)
- moved AIN 1.80 mm to (0.00, 11.4)
- moved AMP1 1.80 mm to (8.89, 7.62)
Routing:
- net AMPVCC: track 31.9 -> 30.1 mm
- net N$53: track 10.7 -> 11.4 mm
Changed lines of the file:
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@@
 <attribute name="VALUE" x="-10.541" y="-0.635" size="1.27" layer="27" ratio="10" rot="R90"/>
 </element>
-<element name="SP+" library="ytani-con-lstb" package="MA02-1" value="" x="2.54" y="1.27" smashed="yes" rot="R90">
-<attribute name="NAME" x="0.889" y="-1.27" size="0.8128" layer="25" ratio="10" rot="R90"/>
-<attribute name="VALUE" x="5.461" y="-1.27" size="1.27" layer="27" ratio="10" rot="R90"/>
-</element>
-<element name="VOL" library="ytani-con-lstb" package="MA02-1" value="" x="2.54" y="6.35" smashed="yes" rot="R90">
-<attribute name="NAME" x="0.889" y="5.08" size="0.8128" layer="25" ratio="10" rot="R90"/>
-<attribute name="VALUE" x="5.461" y="3.81" size="1.27" layer="27" ratio="10" rot="R90"/>
-</element>
-<element name="AIN" library="ytani-con-lstb" package="MA01-1" value="" x="1.27" y="10.16" smashed="yes">
-<attribute name="NAME" x="0.889" y="10.16" size="0.8128" layer="25" ratio="10" rot="R90"/>
-<attribute name="VALUE" x="1.27" y="7.239" size="1.27" layer="27" ratio="10"/>
-</element>
-<element name="AMP1" library="ytani1" package="PAM8012MOD-A" value="" x="10.16" y="6.35" smashed="yes" rot="R270">
-<attribute name="CHIP1" value="PAM8012" x="10.16" y="6.35" size="1.778" layer="27" rot="R270" display="off"/>
-<attribute name="NAME" x="16.51" y="11.43" size="1.778" layer="25" rot="R270"/>
-<attribute name="OC_AKIZUKI" value="K-08217" x="10.16" y="6.35" size="1.778" layer="27" rot="R270" display="off"/>
-<attribute name="URL_AKIZUKI" value="https://akizukidenshi.com/catalog/g/gK-08217/" x="10.16" y="6.35" size="1.778" layer="27" rot="R270" display="off"/>
+<element name="SP+" library="ytani-con-lstb" package="MA02-1" value="" x="1.27" y="2.54" smashed="yes" rot="R90">
+<attribute name="NAME" x="-0.381" y="0" size="0.8128" layer="25" ratio="10" rot="R90"/>
+<attribute name="VALUE" x="4.191" y="0" size="1.27" layer="27" ratio="10" rot="R90"/>
+</element>
+<element name="VOL" library="ytani-con-lstb" package="MA02-1" value="" x="1.27" y="7.62" smashed="yes" rot="R90">
+<attribute name="NAME" x="-0.381" y="6.35" size="0.8128" layer="25" ratio="10" rot="R90"/>
+<attribute name="VALUE" x="4.191" y="5.08" size="1.27" layer="27" ratio="10" rot="R90"/>
+</element>
+<element name="AIN" library="ytani-con-lstb" package="MA01-1" value="" x="0" y="11.43" smashed="yes">
+<attribute name="NAME" x="-0.381" y="11.43" size="0.8128" layer="25" ratio="10" rot="R90"/>
+<attribute name="VALUE" x="0" y="8.509" size="1.27" layer="27" ratio="10"/>
+</element>
+<element name="AMP1" library="ytani1" package="PAM8012MOD-A" value="" x="8.89" y="7.62" smashed="yes" rot="R270">
+<attribute name="CHIP1" value="PAM8012" x="8.89" y="7.62" size="1.778" layer="27" rot="R270" display="off"/>
+<attribute name="NAME" x="15.24" y="12.7" size="1.778" layer="25" rot="R270"/>
+<attribute name="OC_AKIZUKI" value="K-08217" x="8.89" y="7.62" size="1.778" layer="27" rot="R270" display="off"/>
+<attribute name="URL_AKIZUKI" value="https://akizukidenshi.com/catalog/g/gK-08217/" x="8.89" y="7.62" size="1.778" layer="27" rot="R270" display="off"/>
 </element>
 <element name="MD1" library="ytani1" package="DRV8835MOD" value="" x="-16.51" y="-26.67" smashed="yes">
@@
 <wire x1="19.05" y1="26" x2="15.695028125" y2="26" width="0.6096" layer="1"/>
 <wire x1="10.16" y1="21.925" x2="15.695028125" y2="26" width="0.6096" layer="1"/>
-<wire x1="13.97" y1="10.16" x2="13.97" y2="11.43" width="0.6096" layer="1"/>
-<wire x1="13.97" y1="11.43" x2="10.16" y2="15.24" width="0.6096" layer="1"/>
+<wire x1="12.7" y1="11.43" x2="12.7" y2="12.7" width="0.6096" layer="1"/>
+<wire x1="12.7" y1="12.7" x2="10.16" y2="15.24" width="0.6096" layer="1"/>
 <wire x1="10.16" y1="15.24" x2="10.16" y2="21.925" width="0.6096" layer="1"/>
 <wire x1="20.32" y1="25.4" x2="24.13" y2="25.4" width="0.6096" layer="1"/>
@@
 <contactref element="AMP1" pad="SP+@1" route="any" routetag="G$1.SP+"/>
 <contactref element="SP+" pad="1"/>
-<wire x1="11.43" y1="2.54" x2="11.43" y2="1.27" width="0.6096" layer="16"/>
-<wire x1="11.43" y1="1.27" x2="10.16" y2="0" width="0.6096" layer="16"/>
-<wire x1="10.16" y1="0" x2="2.54" y2="0" width="0.6096" layer="16"/>
+<wire x1="10.16" y1="3.81" x2="10.16" y2="1.27" width="0.6096" layer="16"/>
+<wire x1="10.16" y1="1.27" x2="1.27" y2="1.27" width="0.6096" layer="16"/>
 </signal>
 <signal name="N$54">
 <contactref element="AMP1" pad="SP-@1"/>
 <contactref element="SP+" pad="2"/>
-<wire x1="8.89" y1="2.54" x2="2.54" y2="2.54" width="0.6096" layer="16"/>
+<wire x1="7.62" y1="3.81" x2="1.27" y2="3.81" width="0.6096" layer="16"/>
 </signal>
 <signal name="N$56">
 <contactref element="AMP1" pad="IN+"/>
 <contactref element="VOL" pad="1"/>
-<wire x1="2.54" y1="5.08" x2="7.62" y2="5.08" width="0.6096" layer="16"/>
-<wire x1="7.62" y1="5.08" x2="8.89" y2="6.35" width="0.6096" layer="16"/>
-<wire x1="8.89" y1="6.35" x2="8.89" y2="10.16" width="0.6096" layer="16"/>
+<wire x1="1.27" y1="6.35" x2="6.35" y2="6.35" width="0.8128" layer="16"/>
+<wire x1="6.35" y1="6.35" x2="7.62" y2="7.62" width="0.8128" layer="16"/>
+<wire x1="7.62" y1="7.62" x2="7.62" y2="11.43" width="0.8128" layer="16"/>
 </signal>
 <signal name="N$57">
 <contactref element="AIN" pad="1"/>
 <contactref element="VOL" pad="2"/>
-<wire x1="2.54" y1="10.16" x2="2.54" y2="7.62" width="0.8128" layer="16"/>
+<wire x1="1.27" y1="11.43" x2="1.27" y2="8.89" width="0.8128" layer="16"/>
 </signal>
 <signal name="N$50">

Commit message: pcb
Parts:
- removed +5V1: (no value), ytani-con-lstb:MA02-1
- removed R2: (no value), rcl:0204/7
- added JP1: (no value), ytani-con-lstb:MA02-1
- added R1: (no value), rcl:0204/7
- moved +3.3V 9.25 mm to (-6.35, -2.54)
- moved I2C1 6.48 mm to (-14.0, -7.62), turned to 270 degrees
- moved I2C2 6.48 mm to (-10.2, -7.62), turned to 270 degrees
- moved I2C_IN 6.48 mm to (-6.35, -7.62), turned to 90 degrees
- moved MTR_IN 2.84 mm to (-5.08, -24.1)
- moved MTR_OUT 2.54 mm to (-25.4, -21.6)
- moved MD1 1.80 mm to (-15.2, -25.4)
- moved DC-DC_5V 1.28 mm to (-1.27, 23.0)
- moved SV1 1.27 mm to (-21.6, 7.62)
- moved SV5 1.27 mm to (-21.6, -7.62)
- moved SV2 1.27 mm to (-21.6, 3.81)
- moved SV3 1.27 mm to (-21.6, 0.00)
- moved SV4 1.27 mm to (-21.6, -3.81)
- moved +5V 1.27 mm to (19.1, 29.2)
- moved BAT 1.27 mm to (19.1, -29.2), turned to 90 degrees
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- renumbered AIN to AUDIO, AMP1 to AMP
Connections:
- net N$4 renamed BAT+1
- net N$45 renamed SDA
- net N$46 renamed SCL
- net N$5 renamed SDA0
- net N$50 renamed BIN2
- net N$52 renamed BIN1
- net N$53 renamed SP+
- net N$54 renamed SP-
- net N$55 renamed AIN2
- net N$56 renamed AUDIO1
- net N$57 renamed AUDIO0
- net N$58 renamed AIN1
- net N$59 renamed AOUT1
- net N$6 renamed SCL0
- net N$60 renamed AOUT2
- net N$61 renamed BOUT1
- net N$62 renamed BOUT2
- removed net AMPVCC: AMP.V+, RPI1.2, RPI2.2
- removed net N$1: BAT.2, CHG1.BAT+
- removed net N$2: BAT.1, CHG1.BAT-
- new net BAT+0: BAT.1, CHG1.BAT+
- new net BAT+2: JP1.1, SW1.2
- new net BAT-0: BAT.2, CHG1.BAT-
- net +3V3: now also +3.3V.1; no longer +3.3V.2
- net +5V: now also AMP.V+, RPI1.2, RPI2.2; no longer +5V1.1
- net BAT+: now also JP1.2, R1.2; no longer R2.2, SW1.2
- net GND: now also +3.3V.2; no longer +3.3V.1, +5V1.2
- net N$3: now also R1.1; no longer R2.1
Routing:
- net +5V: track 7.33 -> 46.6 mm
- net BAT+0: track 0.00 -> 32.7 mm
- net N$1: track 30.3 -> 0.00 mm
- net AMPVCC: track 30.1 -> 0.00 mm
- net BAT-0: track 0.00 -> 24.8 mm
- net N$2: track 24.0 -> 0.00 mm
- net BAT+2: track 0.00 -> 6.13 mm
- net BAT+1: track 43.6 -> 38.5 mm
- net +3V3: track 57.0 -> 60.8 mm
- net BOUT1: track 4.34 -> 7.62 mm
- net AOUT2: track 4.34 -> 7.62 mm
- net AOUT1: track 4.34 -> 7.62 mm
- net BOUT2: track 4.34 -> 7.62 mm
- net BIN2: track 3.81 -> 5.08 mm
- net BIN1: track 3.81 -> 5.08 mm
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Other:
- outline, holes or cut-outs redrawn
- board text added: "0"
- board text added: "1"
- board text added: "10"
- board text added: "11"
- board text added: "12"
- board text added: "13"
- board text added: "14"
- board text added: "15"
- board text added: "16"
- board text added: "17"
- board text added: "18"
- board text added: "19"
- board text added: "2"
- board text added: "20"
- board text added: "21"
- board text added: "22"
- board text added: "23"
- board text added: "24"
- board text added: "25"
- board text added: "26"
- board text added: "27"
- board text added: "3"
- board text added: "3 V"
- board text added: "3V"
- board text added: "4"
- board text added: "5"
- board text added: "5 V"
- board text added: "6"
- board text added: "7"
- board text added: "8"
- board text added: "9"
- board text added: "G"

Commit message: pcb
Parts:
- removed I2C_IN: (no value), ytani-con-lstb:MA02-1
- added GPIO: (no value), ytani-con-lstb:MA01-1
- added MODE: (no value), ytani-con-lstb:MA03-1
- added R2: 10K, rcl:0204/7
- added SW2: (no value), ytani-con-lstb:MA02-1
- R1: value (none) -> 1K
- moved +3.3V 6.84 mm to (-12.7, 0.00)
- moved AUDIO 5.08 mm to (-5.08, 11.4)
- moved SP+ 5.08 mm to (-3.81, 2.54)
- moved VOL 5.08 mm to (-3.81, 7.62)
- moved I2C1 1.27 mm to (-12.7, -7.62)
- moved MD1 1.27 mm to (-16.5, -25.4)
- moved AMP 1.27 mm to (7.62, 7.62)
- moved DC-DC_5V 1.27 mm to (-2.54, 23.0)
- moved I2C2 1.27 mm to (-8.89, -7.62)
- moved MTR_IN 1.27 mm to (-5.08, -25.4)
- moved MTR_OUT 1.27 mm to (-25.4, -20.3)
- turned +5V to 90 degrees
- turned BAT+ to 90 degrees
- renumbered BAT+1 to BAT+
Connections:
- removed net N$44: RPI1.1, RPI2.1
- removed net SCL0: RPI1.5, RPI2.5
- removed net SDA0: RPI1.3, RPI2.3
- new net MODE: MD1.MODE, MODE.2
- new net N$1: RPI1.17, RPI2.17
- new net N$4: GPIO.1, R2.1, SW2.2
- net +3V3: now also MODE.3, R2.2, RPI1.1, RPI2.1; no longer RPI1.17, RPI2.17
- net GND: now also CHG1.IN-, MODE.1, SW1.3, SW2.1; no longer MD1.MODE
- net SCL: now also RPI1.5, RPI2.5; no longer I2C_IN.1
- net SDA: now also RPI1.3, RPI2.3; no longer I2C_IN.2
Routing:
- net SCL: track 7.62 -> 63.9 mm
- net SDA: track 7.62 -> 60.6 mm
- net +3V3: track 60.8 -> 108.1 mm
- net BAT+1: track 38.5 -> 48.8 mm
- net N$4: track 0.00 -> 7.62 mm
- net MODE: track 0.00 -> 6.88 mm
- net BAT+: track 67.1 -> 61.1 mm
- net N$44: track 5.92 -> 0.00 mm
- net SDA0: track 5.92 -> 0.00 mm
- net SCL0: track 5.92 -> 0.00 mm
- net N$1: track 0.00 -> 5.92 mm
- net SP-: track 6.35 -> 10.2 mm
- net SP+: track 10.7 -> 14.5 mm
- net +5V: track 46.6 -> 43.4 mm
- net AUDIO1: track 11.4 -> 14.5 mm
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Other:
- board text added: "H"
- board text added: "L"
- board text added: "SCL"
- board text added: "SDA"
