File: pcb/OttoPi06a-RPi3AHAT/OttoPi06a-RPi3AHAT.brd (EAGLE design)
At the start: 56 x 65 mm, 31 parts

Commit message: update
Parts:
- removed DCDC1: +5V, ytani1:DCDC-MT3608-MOD2-USB
- added C1: (no value), rcl:C025-024X044
- added DC-DC_5V: (no value), ytani1:DCDC-5V_28V-2A
- moved AMP 2.84 mm to (5.08, 6.35)
- moved R2 2.62 mm to (-0.64, -3.81), turned to 180 degrees
- moved CHG1 1.27 mm to (5.08, -19.0)
- moved MODE 1.27 mm to (-6.35, -17.8)
- moved MTR_IN 1.27 mm to (-6.35, -25.4)
Connections:
- removed net N$17: RPI1.6, RPI2.6
- removed net N$24: RPI1.14, RPI2.14
- removed net N$26: RPI1.20, RPI2.20
- removed net N$40: RPI1.25, RPI2.25
- removed net N$41: RPI1.30, RPI2.30
- removed net N$42: RPI1.34, RPI2.34
- removed net N$8: RPI1.9, RPI2.9
- net +5V: now also DC-DC_5V.VOUT+; no longer DCDC1.VOUT+
- net AUDIO1: now also C1.2
- net BAT+: now also DC-DC_5V.VIN+; no longer DCDC1.VIN+
- net GND: now also C1.1, DC-DC_5V.VIN-, DC-DC_5V.VOUT-, RPI1.14, RPI1.20, RPI1.25, RPI1.30, RPI1.34, RPI1.6, RPI1.9, RPI2.14, RPI2.20, RPI2.25, RPI2.30, RPI2.34, RPI2.6, RPI2.9; no longer DCDC1.VIN-, DCDC1.VOUT-
Routing:
- net GND: track 5.92 -> 48.3 mm
- net N$4: track 7.62 -> 16.4 mm
- net SCL: track 63.9 -> 57.7 mm
- net BAT+1: track 49.8 -> 43.8 mm
- net N$42: track 5.92 -> 0.00 mm
- net N$41: track 5.92 -> 0.00 mm
- net N$8: track 5.92 -> 0.00 mm
- net N$40: track 5.92 -> 0.00 mm
- net N$26: track 5.92 -> 0.00 mm
- net N$24: track 5.92 -> 0.00 mm
- net N$17: track 5.92 -> 0.00 mm
- net SDA: track 60.6 -> 57.4 mm
- net +5V: track 44.4 -> 42.2 mm
- net +3V3: track 108.1 -> 106.0 mm
- net SP+: track 14.5 -> 12.5 mm
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Other:
- board text added: "+V"
- board text added: "DRV8835"
- board text removed: "3V"

Commit message: update
Parts:
- removed DC-DC_5V: (no value), ytani1:DCDC-5V_28V-2A
- added DCDC1: (no value), ytani1:DCDC-MT3608-MOD2-USB
Connections:
- net +5V: now also DCDC1.VOUT+; no longer DC-DC_5V.VOUT+
- net BAT+: now also DCDC1.VIN+; no longer DC-DC_5V.VIN+
- net GND: now also DCDC1.VIN-, DCDC1.VOUT-; no longer DC-DC_5V.VIN-, DC-DC_5V.VOUT-
Other:
- board text added: "OFF"
- board text added: "ON"
Changed lines of the file:
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@@
 <text x="-22.225" y="-13.335" size="0.8128" layer="21" rot="R180">+V</text>
 <text x="-15.24" y="-11.43" size="0.8128" layer="21" rot="R270">G</text>
+<text x="-27.305" y="13.97" size="1.27" layer="21">ON</text>
+<text x="-27.305" y="25.4" size="1.27" layer="21">OFF</text>
 </plain>
 <attributes>
@@
 </autorouter>
 <elements>
-<element name="DC-DC_5V" library="ytani1" package="DCDC-5V_28V-2A" value="" x="-2.54" y="23" smashed="yes">
-<attribute name="NAME" x="-11.43" y="24.27" size="1.27" layer="25"/>
-<attribute name="URL_AMAZON" value="https://www.amazon.co.jp/gp/product/B01D0WSBGY/" x="-2.54" y="23" size="1.778" layer="27" display="off"/>
-<attribute name="VALUE" x="2.54" y="31.89" size="1.778" layer="27"/>
-</element>
 <element name="BAT" library="ytani1" package="JST-PH2" package3d_urn="urn:adsk.eagle:package:23610139/1" value="" x="19.05" y="-29.21" smashed="yes" rot="R90">
 <attribute name="NAME" x="15.24" y="-29.21" size="0.8128" layer="25" rot="R270"/>
@@
 </element>
 <element name="LED1" library="led" library_urn="urn:adsk.eagle:library:259" package="LED3MM" package3d_urn="urn:adsk.eagle:package:15797/1" value="" x="-25.4" y="11.43" smashed="yes" rot="R270">
-<attribute name="NAME" x="-22.86" y="13.97" size="0.8128" layer="25" ratio="10" rot="R270"/>
+<attribute name="NAME" x="-22.86" y="13.335" size="0.8128" layer="25" ratio="10" rot="R270"/>
 <attribute name="POPULARITY" value="97" x="-25.4" y="11.43" size="1.778" layer="27" rot="R270" display="off"/>
 <attribute name="VALUE" x="-27.051" y="9.525" size="1.27" layer="27" ratio="10" rot="R270"/>
@@
 </element>
 <element name="SP+" library="ytani-con-lstb" package="MA02-1" value="" x="-3.81" y="2.54" smashed="yes" rot="R90">
-<attribute name="NAME" x="-1.651" y="0" size="0.8128" layer="25" ratio="10" rot="R90"/>
+<attribute name="NAME" x="-5.08" y="0" size="1.016" layer="25" ratio="10" rot="R90"/>
 <attribute name="VALUE" x="-0.889" y="0" size="1.27" layer="27" ratio="10" rot="R90"/>
 </element>
 <element name="VOL" library="ytani-con-lstb" package="MA02-1" value="" x="-3.81" y="7.62" smashed="yes" rot="R90">
-<attribute name="NAME" x="-1.651" y="6.35" size="0.8128" layer="25" ratio="10" rot="R90"/>
+<attribute name="NAME" x="-5.461" y="6.35" size="0.8128" layer="25" ratio="10" rot="R90"/>
 <attribute name="VALUE" x="-0.889" y="5.08" size="1.27" layer="27" ratio="10" rot="R90"/>
 </element>
 <element name="AUDIO" library="ytani-con-lstb" package="MA01-1" value="" x="-5.08" y="11.43" smashed="yes">
-<attribute name="NAME" x="-1.651" y="10.16" size="0.8128" layer="25" ratio="10" rot="R90"/>
+<attribute name="NAME" x="-5.461" y="10.16" size="0.8128" layer="25" ratio="10" rot="R90"/>
 <attribute name="VALUE" x="-5.08" y="8.509" size="1.27" layer="27" ratio="10"/>
 </element>
@@
 </element>
 <element name="BAT+" library="ytani-con-lstb" package="MA02-1" value="" x="-20.32" y="29.21" smashed="yes" rot="R90">
-<attribute name="NAME" x="-18.161" y="26.67" size="0.8128" layer="25" ratio="10" rot="R90"/>
+<attribute name="NAME" x="-18.161" y="25.4" size="0.8128" layer="25" ratio="10" rot="R90"/>
 <attribute name="VALUE" x="-17.399" y="26.67" size="1.27" layer="27" ratio="10" rot="R90"/>
 </element>
@@
 <attribute name="VALUE" x="6.858" y="15.367" size="1.27" layer="27" ratio="10" rot="R180"/>
 </element>
+<element name="DCDC1" library="ytani1" library_urn="urn:adsk.eagle:library:23610107" package="DCDC-MT3608-MOD2-USB" package3d_urn="urn:adsk.eagle:package:23610144/1" value="" x="-2.54" y="22.86" smashed="yes">
+<attribute name="AMAZON_URL" value="https://www.amazon.co.jp/gp/product/B01D0WSBGY/" x="-2.54" y="22.86" size="1.778" layer="27" display="off"/>
+<attribute name="NAME" x="-17.78" y="31.75" size="1.778" layer="25"/>
+<attribute name="VALUE" x="2.54" y="31.75" size="1.778" layer="27"/>
+</element>
 </elements>
 <signals>
@@
 <contactref element="CHG1" pad="OUT-"/>
 <contactref element="LED1" pad="K"/>
-<contactref element="DC-DC_5V" pad="VIN-"/>
-<contactref element="DC-DC_5V" pad="VOUT-"/>
-<contactref element="+5V" pad="2"/>
 <polygon width="0.15" layer="16">
 <vertex x="-26.67" y="25.4"/>
@@
 <wire x1="23.3409875" y1="20.2112" x2="24.5021875" y2="19.05" width="0.6096" layer="1"/>
 <contactref element="C1" pad="1"/>
+<contactref element="DCDC1" pad="VIN-"/>
+<contactref element="+5V" pad="2"/>
+<contactref element="DCDC1" pad="VOUT-"/>
 </signal>
 <signal name="BAT+">
-<contactref element="DC-DC_5V" pad="VIN+"/>
 <contactref element="R1" pad="2"/>
 <contactref element="BAT+" pad="1"/>
@@
 <wire x1="-21.59" y1="-15.24" x2="-19.05" y2="-15.24" width="0.8128" layer="1"/>
 <contactref element="JP1" pad="2"/>
-<wire x1="-20.32" y1="25.4" x2="-17.78" y2="25.4" width="0.8128" layer="1"/>
-<wire x1="-17.78" y1="20.32" x2="-17.78" y2="25.4" width="0.8128" layer="1"/>
 <wire x1="-17.78" y1="11.43" x2="-19.05" y2="10.16" width="0.8128" layer="1"/>
 <wire x1="-19.05" y1="10.16" x2="-21.59" y2="10.16" width="0.8128" layer="1"/>
@@
 <wire x1="-17.78" y1="20.32" x2="-17.78" y2="11.43" width="0.8128" layer="1"/>
 <wire x1="-22.86" y1="8.89" x2="-22.86" y2="7.62" width="0.8128" layer="1"/>
-<wire x1="-15.79" y1="26.12" x2="-15.79" y2="30" width="0.8128" layer="1"/>
-<wire x1="-20.32" y1="25.4" x2="-20.32" y2="27.94" width="0.6096" layer="1"/>
-<wire x1="-15.79" y1="26.12" x2="-16.51" y2="25.4" width="0.8128" layer="1"/>
-<wire x1="-16.51" y1="25.4" x2="-17.78" y2="25.4" width="0.8128" layer="1"/>
+<contactref element="DCDC1" pad="VIN+"/>
+<wire x1="-15.79" y1="27.94" x2="-15.79" y2="29.86" width="0.8128" layer="1"/>
+<wire x1="-20.32" y1="27.94" x2="-17.78" y2="27.94" width="0.8128" layer="1"/>
+<wire x1="-17.78" y1="27.94" x2="-15.79" y2="27.94" width="0.8128" layer="1"/>
+<wire x1="-17.78" y1="20.32" x2="-17.78" y2="27.94" width="0.8128" layer="1"/>
+<wire x1="-20.32" y1="25.4" x2="-20.32" y2="26.67" width="0.8128" layer="1"/>
+<wire x1="-20.32" y1="26.67" x2="-20.32" y2="27.94" width="0.8128" layer="1"/>
+<wire x1="-20.32" y1="26.67" x2="-20.32" y2="26.67" width="0.8128" layer="1"/>
 </signal>
 <signal name="+5V">
-<contactref element="DC-DC_5V" pad="VOUT+"/>
 <contactref element="+5V" pad="1"/>
 <contactref element="RPI2" pad="2"/>
@@
 <wire x1="24.6474" y1="26.1526" x2="20.32" y2="26.1526" width="0.8128" layer="1"/>
 <wire x1="20.32" y1="24.13" x2="20.32" y2="26.1526" width="0.8128" layer="1"/>
-<wire x1="10.71" y1="30" x2="10.71" y2="28.66" width="0.8128" layer="1"/>
-<wire x1="10.71" y1="28.66" x2="11.43" y2="27.94" width="0.8128" layer="1"/>
+<wire x1="11.43" y1="27.94" x2="10.71" y2="28.66" width="0.8128" layer="1"/>
 <wire x1="11.43" y1="27.94" x2="19.05" y2="27.94" width="0.8128" layer="1"/>
 <contactref element="AMP" pad="V+"/>
-<wire x1="8.17" y1="27.46" x2="10.71" y2="30" width="0.8128" layer="16"/>
 <wire x1="8.89" y1="10.16" x2="8.89" y2="13.97" width="0.8128" layer="16"/>
 <wire x1="8.89" y1="13.97" x2="8.17" y2="14.69" width="0.8128" layer="16"/>
 <wire x1="8.17" y1="14.69" x2="8.17" y2="27.46" width="0.8128" layer="16"/>
+<contactref element="DCDC1" pad="VOUT+"/>
+<wire x1="8.17" y1="27.46" x2="10.57" y2="29.86" width="0.8128" layer="16"/>
+<wire x1="10.57" y1="29.86" x2="10.71" y2="29.86" width="0.8128" layer="16"/>
+<wire x1="10.71" y1="28.66" x2="10.71" y2="29.86" width="0.8128" layer="1"/>
 </signal>
 <signal name="BAT+1">

Commit message: pcb
Parts:
- added JP2: (no value), ytani1:PINHEAD-MA02-1
- added SV7, SV8, SV9: (no value), ytani1:PINHEAD-MA04-1
- +3.3V, +5V, BAT+, JP1, SP+, SW2, VOL: device ytani-con-lstb:MA02-1 -> ytani1:PINHEAD-MA02-1
- AUDIO, GPIO: device ytani-con-lstb:MA01-1 -> ytani1:PINHEAD-MA01-1
- I2C1, I2C2, MTR_IN, MTR_OUT, SV1, SV2, SV3, SV4, SV5, SV6: device ytani-con-lstb:MA04-1 -> ytani1:PINHEAD-MA04-1
- MODE: device ytani-con-lstb:MA03-1 -> ytani1:PINHEAD-MA03-1
- moved R2 12.0 mm to (-10.8, 2.54), turned to 270 degrees
- moved SV6 5.71 mm to (-21.6, -5.71)
- moved GPIO 5.12 mm to (-14.6, 1.27)
- moved SW2 5.12 mm to (-13.3, 5.08)
- moved SV5 4.45 mm to (-21.6, -3.17)
- moved +5V 3.86 mm to (15.2, 28.6), turned to 270 degrees
- moved AMP 3.81 mm to (1.27, 6.35)
- moved C1 3.81 mm to (1.27, 12.7)
- moved SV4 3.17 mm to (-21.6, -0.64)
- moved +3.3V 2.62 mm to (-13.3, -2.54)
- moved AUDIO 2.62 mm to (-7.62, 10.8)
- moved SP+ 2.62 mm to (-6.35, 1.91)
- moved VOL 2.62 mm to (-6.35, 6.99)
- moved SV3 1.91 mm to (-21.6, 1.91)
- moved I2C1 1.90 mm to (-10.8, -7.62)
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Connections:
- new net N$2: SV7.3, SV7.4
- new net N$5: SV8.3, SV8.4
- new net N$6: JP2.2, RPI1.2, RPI2.2
- new net N$8: SV9.3, SV9.4
- net +5V: now also JP2.1; no longer AMP.V+, RPI1.2, RPI2.2
- net BAT+: now also AMP.V+, SV7.2, SV8.2, SV9.2
- net GND: now also SV7.1, SV8.1, SV9.1
Routing:
- net +5V: track 42.0 -> 7.08 mm
- net BAT+: track 61.4 -> 90.5 mm
- net +3V3: track 106.0 -> 80.6 mm
- net N$6: track 0.00 -> 12.0 mm
- net N$4: track 16.4 -> 7.62 mm
- net N$8: track 0.00 -> 2.54 mm
- net N$5: track 0.00 -> 2.54 mm
- net N$2: track 0.00 -> 2.54 mm
- net SP+: track 12.5 -> 10.4 mm
- net BAT+0: track 33.9 -> 32.1 mm
- net BAT+1: track 43.8 -> 42.2 mm
- net SP-: track 8.15 -> 6.61 mm
- net SCL: track 57.7 -> 57.1 mm
Other:
- board text added: "3V"
- board text added: "VM"
- board text removed: "+V"
- board text removed: "3 V"

Commit message: pcb
Parts:
- moved I2C1 0.90 mm to (-11.4, -8.26)
- moved I2C2 0.90 mm to (-8.89, -8.26)
- moved GPIO 0.90 mm to (-15.2, 0.64)
- moved R2 0.90 mm to (-11.4, 1.91)
- moved +3.3V 0.90 mm to (-14.0, -3.17)
- moved SW2 0.90 mm to (-14.0, 4.45)
- moved R1 0.63 mm to (-21.0, 16.5)
Routing:
- net BAT+1: track 42.2 -> 44.4 mm
- net BAT+: track 90.5 -> 89.4 mm
- net N$3: track 5.08 -> 4.45 mm
