File: pcb/OttoPi06a-RPi3AHAT/OttoPi06a-RPi3AHAT.sch (EAGLE design)
At the start: 28 parts

Commit message: pcb
Parts:
- removed +5V1: (no value), ytani-con-lstb:MA02-1
- removed R2: (no value), rcl:R-US_0204/7
- added JP1: (no value), ytani-con-lstb:MA02-1
- added R1: (no value), rcl:R-US_0204/7
- renumbered AIN to AUDIO, AMP1 to AMP
Connections:
- net N$4 renamed BAT+1
- net N$45 renamed SDA
- net N$46 renamed SCL
- net N$5 renamed SDA0
- net N$50 renamed BIN2
- net N$52 renamed BIN1
- net N$53 renamed SP+
- net N$54 renamed SP-
- net N$55 renamed AIN2
- net N$56 renamed AUDIO1
- net N$57 renamed AUDIO0
- net N$58 renamed AIN1
- net N$59 renamed AOUT1
- net N$6 renamed SCL0
- net N$60 renamed AOUT2
- net N$61 renamed BOUT1
- net N$62 renamed BOUT2
- removed net AMPVCC: AMP.VCC, RPI1.5V@1, RPI2.5V@1
- removed net N$1: BAT.2, CHG1.BAT+
- removed net N$2: BAT.1, CHG1.BAT-
- new net BAT+0: BAT.1, CHG1.BAT+
- new net BAT+2: JP1.1, SW1.2
- new net BAT-0: BAT.2, CHG1.BAT-
- net +3V3: now also +3.3V.1; no longer +3.3V.2
- net +5V: now also AMP.VCC, RPI1.5V@1, RPI2.5V@1; no longer +5V1.1
- net BAT+: now also JP1.2, R1.2; no longer R2.2, SW1.2
- net GND: now also +3.3V.2; no longer +3.3V.1, +5V1.2
- net N$3: now also R1.1; no longer R2.1
Other:
- moved on the sheet: +3.3V, +5V, BAT, BAT+1, CHG1, DC-DC_5V, LED1, MD1, MTR_IN, MTR_OUT

Commit message: pcb
Parts:
- removed BAT+1, I2C_IN: (no value), ytani-con-lstb:MA02-1
- added BAT+, SW2: (no value), ytani-con-lstb:MA02-1
- added GPIO: (no value), ytani-con-lstb:MA01-1
- added MODE: (no value), ytani-con-lstb:MA03-1
- added R2: 10K, rcl:R-US_0204/7
- R1: value (none) -> 1K
Connections:
- removed net N$44: RPI1.3V3@1, RPI2.3V3@1
- removed net SCL0: RPI1.GPIO3(SCL), RPI2.GPIO3(SCL)
- removed net SDA0: RPI1.GPIO2(SDA), RPI2.GPIO2(SDA)
- new net MODE: MD1.MODE, MODE.2
- new net N$1: RPI1.3V3@2, RPI2.3V3@2
- new net N$4: GPIO.1, R2.1, SW2.2
- net +3V3: now also MODE.3, R2.2, RPI1.3V3@1, RPI2.3V3@1; no longer RPI1.3V3@2, RPI2.3V3@2
- net BAT+: now also BAT+.1; no longer BAT+1.1
- net GND: now also BAT+.2, CHG1.IN-, MODE.1, SW1.3, SW2.1; no longer BAT+1.2, MD1.MODE
- net SCL: now also RPI1.GPIO3(SCL), RPI2.GPIO3(SCL); no longer I2C_IN.1
- net SDA: now also RPI1.GPIO2(SDA), RPI2.GPIO2(SDA); no longer I2C_IN.2
Other:
- moved on the sheet: +3.3V, +5V, AMP, AUDIO, BAT, CHG1, DC-DC_5V, I2C1, I2C2, JP1, LED1, MD1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
