File: pcb/OttoPi06a-RPi3AHAT/OttoPi06a-RPi3AHAT.sch (EAGLE design)
At the start: 31 parts

Commit message: update
Parts:
- added C1: (no value), rcl:C-EU025-024X044
Connections:
- removed net N$17: RPI1.GND@1, RPI2.GND@1
- removed net N$24: RPI1.GND@3, RPI2.GND@3
- removed net N$26: RPI1.GND@4, RPI2.GND@4
- removed net N$40: RPI1.GND@5, RPI2.GND@5
- removed net N$41: RPI1.GND@6, RPI2.GND@6
- removed net N$42: RPI1.GND@7, RPI2.GND@7
- removed net N$8: RPI1.GND@2, RPI2.GND@2
- net AUDIO1: now also C1.2
- net GND: now also C1.1, RPI1.GND@1, RPI1.GND@2, RPI1.GND@3, RPI1.GND@4, RPI1.GND@5, RPI1.GND@6, RPI1.GND@7, RPI2.GND@1, RPI2.GND@2, RPI2.GND@3, RPI2.GND@4, RPI2.GND@5, RPI2.GND@6, RPI2.GND@7
Other:
- moved on the sheet: AMP, AUDIO, SP+, VOL

Commit message: update
Parts:
- removed DC-DC_5V: (no value), ytani1:DCDC-5V_28V-2A
- added DCDC1: (no value), ytani1:DCDC-MT3608-MODUSB
Connections:
- net +5V: now also DCDC1.VOUT+; no longer DC-DC_5V.VOUT+
- net BAT+: now also DCDC1.VIN+; no longer DC-DC_5V.VIN+
- net GND: now also DCDC1.VIN-, DCDC1.VOUT-; no longer DC-DC_5V.VIN-, DC-DC_5V.VOUT-
Changed lines of the file:
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@@
 <setting verticaltext="up"/>
 </settings>
-<grid distance="0.635" unitdist="mm" unit="mm" style="lines" multiple="4" display="yes" altdistance="0.01" altunitdist="inch" altunit="inch"/>
+<grid distance="1.27" unitdist="mm" unit="mm" style="lines" multiple="2" display="yes" altdistance="0.01" altunitdist="inch" altunit="inch"/>
 <layers>
 <layer number="1" name="Top" color="4" fill="1" visible="no" active="no"/>
@@
 <part name="GND3" library="supply1" library_urn="urn:adsk.eagle:library:371" deviceset="GND" device=""/>
 <part name="+3V2" library="supply1" library_urn="urn:adsk.eagle:library:371" deviceset="+3V3" device=""/>
-<part name="DC-DC_5V" library="ytani1" deviceset="DCDC-5V_28V-2A" device=""/>
 <part name="BAT" library="ytani1" deviceset="JST-PH2" device="" package3d_urn="urn:adsk.eagle:package:23610139/1"/>
 <part name="CHG1" library="ytani1" deviceset="TP4056MOD1" device="" package3d_urn="urn:adsk.eagle:package:23610133/1"/>
@@
 <part name="LED1" library="led" library_urn="urn:adsk.eagle:library:259" deviceset="LED" device="3MM" package3d_urn="urn:adsk.eagle:package:15797/1"/>
 <part name="GND4" library="supply1" library_urn="urn:adsk.eagle:library:371" deviceset="GND" device=""/>
-<part name="GND5" library="supply1" library_urn="urn:adsk.eagle:library:371" deviceset="GND" device=""/>
 <part name="R1" library="rcl" library_urn="urn:adsk.eagle:library:334" deviceset="R-US_" device="0204/7" package3d_urn="urn:adsk.eagle:package:23498/2" value="1K"/>
 <part name="+5V" library="ytani-con-lstb" deviceset="MA02-1" device=""/>
@@
 <part name="GND16" library="supply1" library_urn="urn:adsk.eagle:library:371" deviceset="GND" device=""/>
 <part name="C1" library="rcl" library_urn="urn:adsk.eagle:library:334" deviceset="C-EU" device="025-024X044" package3d_urn="urn:adsk.eagle:package:23630/1"/>
+<part name="DCDC1" library="ytani1" library_urn="urn:adsk.eagle:library:23610107" deviceset="DCDC-MT3608-MOD" device="USB" package3d_urn="urn:adsk.eagle:package:23610144/1"/>
+<part name="GND5" library="supply1" library_urn="urn:adsk.eagle:library:371" deviceset="GND" device=""/>
 </parts>
 <sheets>
@@
 <attribute name="VALUE" x="-55.88" y="99.06" size="1.778" layer="96"/>
 </instance>
-<instance part="DC-DC_5V" gate="G$1" x="27.94" y="142.24" smashed="yes">
-<attribute name="NAME" x="17.78" y="147.32" size="1.778" layer="95"/>
-<attribute name="VALUE" x="38.32" y="143.24" size="1.4224" layer="96"/>
-</instance>
 <instance part="BAT" gate="G$1" x="-17.78" y="177.8" smashed="yes">
 <attribute name="NAME" x="-22.86" y="181.102" size="1.778" layer="95"/>
@@
 <attribute name="VALUE" x="-2.54" y="114.3" size="1.778" layer="96"/>
 </instance>
-<instance part="GND5" gate="1" x="43.18" y="116.84" smashed="yes">
-<attribute name="VALUE" x="40.64" y="114.3" size="1.778" layer="96"/>
-</instance>
 <instance part="R1" gate="G$1" x="0" y="137.16" smashed="yes" rot="R90">
 <attribute name="NAME" x="-1.4986" y="133.35" size="1.778" layer="95" rot="R90"/>
@@
 <attribute name="NAME" x="82.296" y="63.119" size="1.778" layer="95" rot="R180"/>
 <attribute name="VALUE" x="82.296" y="68.199" size="1.778" layer="96" rot="R180"/>
+</instance>
+<instance part="DCDC1" gate="G$1" x="27.94" y="142.24" smashed="yes">
+<attribute name="NAME" x="17.78" y="147.32" size="1.778" layer="95"/>
+<attribute name="VALUE" x="38.32" y="143.24" size="1.4224" layer="96"/>
+</instance>
+<instance part="GND5" gate="1" x="43.18" y="116.84" smashed="yes">
+<attribute name="VALUE" x="40.64" y="114.3" size="1.778" layer="96"/>
 </instance>
 </instances>
@@
 <segment>
 <wire x1="12.7" y1="119.38" x2="12.7" y2="139.7" width="0.1524" layer="91"/>
-<wire x1="12.7" y1="139.7" x2="15.24" y2="139.7" width="0.1524" layer="91"/>
-<pinref part="DC-DC_5V" gate="G$1" pin="VIN-"/>
 <pinref part="GND2" gate="1" pin="GND"/>
-</segment>
-<segment>
-<wire x1="43.18" y1="139.7" x2="43.18" y2="119.38" width="0.1524" layer="91"/>
-<wire x1="40.64" y1="139.7" x2="43.18" y2="139.7" width="0.1524" layer="91"/>
-<pinref part="DC-DC_5V" gate="G$1" pin="VOUT-"/>
-<pinref part="GND5" gate="1" pin="GND"/>
-<pinref part="+5V" gate="G$1" pin="2"/>
-<wire x1="45.72" y1="142.24" x2="43.18" y2="142.24" width="0.1524" layer="91"/>
-<wire x1="43.18" y1="142.24" x2="43.18" y2="139.7" width="0.1524" layer="91"/>
-<junction x="43.18" y="139.7"/>
+<pinref part="DCDC1" gate="G$1" pin="VIN-"/>
+<wire x1="15.24" y1="139.7" x2="12.7" y2="139.7" width="0.1524" layer="91"/>
 </segment>
 <segment>
@@
 <junction x="50.8" y="63.5"/>
 </segment>
+<segment>
+<wire x1="43.18" y1="142.24" x2="43.18" y2="139.7" width="0.1524" layer="91"/>
+<pinref part="+5V" gate="G$1" pin="2"/>
+<wire x1="45.72" y1="142.24" x2="43.18" y2="142.24" width="0.1524" layer="91"/>
+<pinref part="DCDC1" gate="G$1" pin="VOUT-"/>
+<wire x1="40.64" y1="139.7" x2="43.18" y2="139.7" width="0.1524" layer="91"/>
+<pinref part="GND5" gate="1" pin="GND"/>
+<wire x1="43.18" y1="119.38" x2="43.18" y2="139.7" width="0.1524" layer="91"/>
+<junction x="43.18" y="139.7"/>
+</segment>
 </net>
 <net name="BAT+" class="0">
@@
 <wire x1="0" y1="180.34" x2="0" y2="175.26" width="0.1524" layer="91"/>
 <wire x1="0" y1="175.26" x2="0" y2="144.78" width="0.1524" layer="91"/>
-<wire x1="0" y1="144.78" x2="15.24" y2="144.78" width="0.1524" layer="91"/>
-<pinref part="DC-DC_5V" gate="G$1" pin="VIN+"/>
 <junction x="0" y="144.78"/>
 <wire x1="0" y1="142.24" x2="0" y2="144.78" width="0.1524" layer="91"/>
@@
 <wire x1="-7.62" y1="144.78" x2="0" y2="144.78" width="0.1524" layer="91"/>
 <junction x="0" y="144.78"/>
+<pinref part="DCDC1" gate="G$1" pin="VIN+"/>
+<wire x1="15.24" y1="144.78" x2="0" y2="144.78" width="0.1524" layer="91"/>
 </segment>
 <segment>
@@
 <pinref part="P+2" gate="1" pin="+5V"/>
 <wire x1="43.18" y1="149.86" x2="43.18" y2="144.78" width="0.1524" layer="91"/>
-<wire x1="43.18" y1="144.78" x2="40.64" y2="144.78" width="0.1524" layer="91"/>
-<pinref part="DC-DC_5V" gate="G$1" pin="VOUT+"/>
 <pinref part="+5V" gate="G$1" pin="1"/>
 <wire x1="43.18" y1="144.78" x2="45.72" y2="144.78" width="0.1524" layer="91"/>
+<pinref part="DCDC1" gate="G$1" pin="VOUT+"/>
+<wire x1="40.64" y1="144.78" x2="43.18" y2="144.78" width="0.1524" layer="91"/>
 <junction x="43.18" y="144.78"/>
 </segment>

Commit message: pcb
Parts:
- added JP2: (no value), ytani1:PINHEAD-MA02-1
- added SV7, SV8, SV9: (no value), ytani1:PINHEAD-MA04-1
- +3.3V, +5V, BAT+, JP1, SP+, SW2, VOL: device ytani-con-lstb:MA02-1 -> ytani1:PINHEAD-MA02-1
- AUDIO, GPIO: device ytani-con-lstb:MA01-1 -> ytani1:PINHEAD-MA01-1
- I2C1, I2C2, MTR_IN, MTR_OUT, SV1, SV2, SV3, SV4, SV5, SV6: device ytani-con-lstb:MA04-1 -> ytani1:PINHEAD-MA04-1
- MODE: device ytani-con-lstb:MA03-1 -> ytani1:PINHEAD-MA03-1
Connections:
- new net N$2: SV7.3, SV7.4
- new net N$5: SV8.3, SV8.4
- new net N$6: JP2.2, RPI1.5V@1, RPI2.5V@1
- new net N$8: SV9.3, SV9.4
- net +5V: now also JP2.1; no longer AMP.VCC, RPI1.5V@1, RPI2.5V@1
- net BAT+: now also AMP.VCC, SV7.2, SV8.2, SV9.2
- net GND: now also SV7.1, SV8.1, SV9.1
Other:
- moved on the sheet: MODE, SV1, SV2, SV3, SV4, SV5, SV6
