File: pcb/OttoPi08-RPi3AHAT/OttoPi08-RPi3AHAT.brd (EAGLE design)
At the start: 56 x 65 mm, 39 parts

Commit message: UPD: pcb/OttoPi08-RPi3AHAT
Parts:
- moved C1 26.4 mm to (-14.6, 13.3), turned to 0 degrees
- moved C2 24.8 mm to (-9.53, 13.3), turned to 0 degrees
- moved AMP 15.3 mm to (-12.1, 20.3), turned to 90 degrees
- moved JP1 5.85 mm to (-20.3, 28.6), turned to 270 degrees
- moved +5V 2.29 mm to (15.9, 28.6), turned to 270 degrees
- moved JP2 1.42 mm to (18.4, 28.6), turned to 270 degrees
- moved AUDIO 1.27 mm to (-5.08, 31.1)
- moved BAT+ 1.27 mm to (-17.8, 28.6), turned to 90 degrees
- moved SP+ 1.27 mm to (-14.0, 29.8)
- moved VOL 1.27 mm to (-8.89, 29.8)
- moved R2 0.90 mm to (-6.99, 3.17)
- moved GPIO 0.90 mm to (-6.99, 10.8)
- moved 3V3 0.90 mm to (-12.1, 3.17)
- moved SW2 0.90 mm to (-10.8, 9.53)
- moved I2C3 0.64 mm to (-6.99, -6.35)
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Routing:
- net SP+: track 17.4 -> 6.50 mm
- net BAT+: track 99.4 -> 92.5 mm
- net SP-: track 13.3 -> 6.50 mm
- net BAT+2: track 5.61 -> 12.2 mm
- net N$15: track 21.2 -> 18.9 mm
- net N$6: track 13.9 -> 11.7 mm
- net SDA: track 53.7 -> 54.8 mm
- net SCL: track 58.1 -> 58.7 mm

Commit message: UPD: pcb/OttoPi08-RPi3AHAT
Parts:
- added DCDC1: (no value), ytani1:DCDC-MT3608-MOD1
- added DCDC3: (no value), ytani1:DCDC-MT3608-MOD2-USB
- moved DCDC2 5.08 mm to (4.45, 11.4)
Connections:
- net +5V: now also DCDC1.VOUT+, DCDC3.VOUT+
- net BAT+: now also DCDC1.VIN+, DCDC3.VIN+
- net GND: now also DCDC1.VIN-, DCDC1.VOUT-, DCDC3.VIN-, DCDC3.VOUT-
Routing:
- net BAT+: track 92.5 -> 102.5 mm
- net SDA: track 54.8 -> 61.1 mm
- net +3V3: track 79.7 -> 84.9 mm
- net SCL: track 58.7 -> 62.1 mm
- net +5V: track 26.3 -> 29.0 mm
Changed lines of the file:
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@@
 <attribute name="VALUE" x="-20.955" y="-11.049" size="1.27" layer="27" ratio="10"/>
 </element>
-<element name="DCDC2" library="ytani1" package="DCDC-SX1308-MOD1" value="" x="4.445" y="6.35" smashed="yes" rot="R90">
-<attribute name="AMAZON_URL" value="https://www.amazon.co.jp/gp/product/B095YKY29M/" x="4.445" y="6.35" size="1.778" layer="27" rot="R90" display="off"/>
-<attribute name="NAME" x="1.905" y="4.445" size="0.8128" layer="25" rot="R90"/>
-<attribute name="VALUE" x="-4.445" y="8.255" size="1.778" layer="27" rot="R90"/>
+<element name="DCDC2" library="ytani1" package="DCDC-SX1308-MOD1" value="" x="4.445" y="11.43" smashed="yes" rot="R90">
+<attribute name="AMAZON_URL" value="https://www.amazon.co.jp/gp/product/B095YKY29M/" x="4.445" y="11.43" size="1.778" layer="27" rot="R90" display="off"/>
+<attribute name="NAME" x="1.905" y="9.525" size="0.8128" layer="25" rot="R90"/>
+<attribute name="VALUE" x="-4.445" y="13.335" size="1.778" layer="27" rot="R90"/>
+</element>
+<element name="DCDC1" library="ytani1" library_urn="urn:adsk.eagle:library:30941153" package="DCDC-MT3608-MOD1" package3d_urn="urn:adsk.eagle:package:23610132/1" value="" x="5.08" y="13.335" smashed="yes" rot="R270">
+<attribute name="AMAZON_URL" value="https://www.amazon.co.jp/gp/product/B086GDTYDS/" x="5.08" y="13.335" size="1.778" layer="27" rot="R270" display="off"/>
+<attribute name="VALUE" x="13.97" y="8.255" size="1.778" layer="27" rot="R270"/>
+</element>
+<element name="DCDC3" library="ytani1" library_urn="urn:adsk.eagle:library:30941153" package="DCDC-MT3608-MOD2-USB" package3d_urn="urn:adsk.eagle:package:23610144/1" value="" x="4.445" y="12.7" smashed="yes" rot="R90">
+<attribute name="AMAZON_URL" value="https://www.amazon.co.jp/gp/product/B01D0WSBGY/" x="4.445" y="12.7" size="1.778" layer="27" rot="R90" display="off"/>
+<attribute name="VALUE" x="-4.445" y="17.78" size="1.778" layer="27" rot="R90"/>
 </element>
 </elements>
@@
 <contactref element="+5V" pad="2"/>
 <contactref element="DCDC2" pad="VOUT-"/>
+<contactref element="DCDC1" pad="VOUT-"/>
+<contactref element="DCDC3" pad="VOUT-"/>
+<contactref element="DCDC1" pad="VIN-"/>
+<contactref element="DCDC3" pad="VIN-"/>
 </signal>
 <signal name="BAT+" class="1">
@@
 <wire x1="-22.225" y1="11.43" x2="-22.225" y2="19.05" width="0.8128" layer="1"/>
 <contactref element="DCDC2" pad="VIN+"/>
-<wire x1="-0.805" y1="-2.9" x2="-0.805" y2="10.965" width="0.8128" layer="16"/>
+<wire x1="-0.805" y1="2.18" x2="-0.805" y2="10.965" width="0.8128" layer="16"/>
 <wire x1="-20.32" y1="20.32" x2="-15.875" y2="20.32" width="0.8128" layer="16"/>
 <wire x1="-15.875" y1="20.32" x2="-15.875" y2="16.51" width="0.8128" layer="16"/>
@@
 <wire x1="-17.78" y1="27.305" x2="-20.32" y2="27.305" width="0.8128" layer="16"/>
 <wire x1="-20.32" y1="20.32" x2="-20.32" y2="27.305" width="0.8128" layer="16"/>
+<contactref element="DCDC3" pad="VIN+"/>
+<contactref element="DCDC1" pad="VIN+"/>
+<wire x1="8.58" y1="-1.665" x2="8.34" y2="-1.905" width="0.8128" layer="16"/>
+<wire x1="5.715" y1="-1.905" x2="3.175" y2="0.635" width="0.8128" layer="16"/>
+<wire x1="3.175" y1="0.635" x2="0" y2="0.635" width="0.8128" layer="16"/>
+<wire x1="-0.805" y1="1.44" x2="-0.805" y2="2.18" width="0.8128" layer="16"/>
+<wire x1="8.34" y1="-1.905" x2="5.715" y2="-1.905" width="0.8128" layer="16"/>
+<wire x1="0" y1="0.635" x2="-0.805" y2="1.44" width="0.8128" layer="16"/>
+<wire x1="-2.555" y1="-0.55" x2="-0.805" y2="1.2" width="0.8128" layer="16"/>
+<wire x1="-0.805" y1="1.2" x2="-0.805" y2="2.18" width="0.8128" layer="16"/>
 </signal>
 <signal name="+5V">
@@
 <contactref element="DCDC2" pad="VOUT+"/>
 <wire x1="15.875" y1="29.845" x2="18.415" y2="29.845" width="0.8128" layer="16"/>
-<wire x1="15.875" y1="29.845" x2="11.43" y2="29.845" width="0.8128" layer="16"/>
-<wire x1="11.43" y1="29.845" x2="-0.805" y2="17.61" width="0.8128" layer="16"/>
-<wire x1="-0.805" y1="15.6" x2="-0.805" y2="17.61" width="0.8128" layer="16"/>
+<contactref element="DCDC1" pad="VOUT+"/>
+<contactref element="DCDC3" pad="VOUT+"/>
+<wire x1="-0.805" y1="20.68" x2="-0.805" y2="21.125" width="0.8128" layer="16"/>
+<wire x1="-2.555" y1="22.875" x2="-2.555" y2="25.95" width="0.8128" layer="16"/>
+<wire x1="-0.805" y1="21.125" x2="-2.555" y2="22.875" width="0.8128" layer="16"/>
+<wire x1="-2.555" y1="25.95" x2="6.9" y2="25.95" width="0.8128" layer="16"/>
+<wire x1="8.58" y1="27.63" x2="8.58" y2="28.335" width="0.8128" layer="16"/>
+<wire x1="6.9" y1="25.95" x2="8.58" y2="27.63" width="0.8128" layer="16"/>
+<wire x1="8.58" y1="28.335" x2="11.19" y2="28.335" width="0.8128" layer="16"/>
+<wire x1="12.7" y1="29.845" x2="15.875" y2="29.845" width="0.8128" layer="16"/>
+<wire x1="11.19" y1="28.335" x2="12.7" y2="29.845" width="0.8128" layer="16"/>
 </signal>
 <signal name="BAT+1">
 <contactref element="CHG1" pad="OUT+"/>
 <contactref element="SW1" pad="1"/>
-<wire x1="-3.81" y1="-5.61" x2="-3.81" y2="9.525" width="0.8128" layer="16"/>
-<wire x1="-3.81" y1="9.525" x2="-5.715" y2="11.43" width="0.8128" layer="16"/>
-<wire x1="-1.82" y1="-7.6" x2="-3.81" y2="-5.61" width="0.8128" layer="16"/>
+<wire x1="-4.445" y1="-4.975" x2="-4.445" y2="10.16" width="0.8128" layer="16"/>
+<wire x1="-4.445" y1="10.16" x2="-5.715" y2="11.43" width="0.8128" layer="16"/>
+<wire x1="-1.82" y1="-7.6" x2="-4.445" y2="-4.975" width="0.8128" layer="16"/>
 <wire x1="-16.51" y1="11.43" x2="-18.415" y2="13.335" width="0.8128" layer="16"/>
 <wire x1="-18.415" y1="13.335" x2="-18.415" y2="15.24" width="0.8128" layer="16"/>
@@
 <wire x1="-13.335" y1="-2.54" x2="-12.065" y2="-2.54" width="0.8128" layer="1"/>
 <wire x1="-12.065" y1="-2.54" x2="-12.065" y2="1.905" width="0.8128" layer="1"/>
-<wire x1="5.08" y1="15.875" x2="5.08" y2="6.35" width="0.8128" layer="1"/>
-<wire x1="5.08" y1="6.35" x2="-1.905" y2="-0.635" width="0.8128" layer="1"/>
-<wire x1="-1.905" y1="-0.635" x2="-6.985" y2="-0.635" width="0.8128" layer="1"/>
-<wire x1="15.875" y1="24.13" x2="13.335" y2="24.13" width="0.8128" layer="1"/>
-<wire x1="13.335" y1="24.13" x2="5.08" y2="15.875" width="0.8128" layer="1"/>
+<wire x1="5.08" y1="20.955" x2="5.08" y2="5.08" width="0.8128" layer="1"/>
+<wire x1="5.08" y1="5.08" x2="-3.81" y2="5.08" width="0.8128" layer="1"/>
+<wire x1="-3.81" y1="5.08" x2="-6.985" y2="1.905" width="0.8128" layer="1"/>
+<wire x1="-6.985" y1="1.905" x2="-6.985" y2="-0.635" width="0.8128" layer="1"/>
+<wire x1="15.875" y1="24.13" x2="8.255" y2="24.13" width="0.8128" layer="1"/>
+<wire x1="8.255" y1="24.13" x2="5.08" y2="20.955" width="0.8128" layer="1"/>
 <wire x1="-6.985" y1="-0.635" x2="-6.985" y2="-2.54" width="0.8128" layer="1"/>
 </signal>
@@
 <wire x1="16.76263125" y1="21.59" x2="17.93103125" y2="22.7584" width="0.6096" layer="16"/>
 <wire x1="18.89896875" y1="22.7584" x2="20.06736875" y2="21.59" width="0.6096" layer="16"/>
-<wire x1="-6.985" y1="-5.08" x2="1.27" y2="-5.08" width="0.8128" layer="1"/>
-<wire x1="12.065" y1="5.715" x2="12.065" y2="19.05" width="0.8128" layer="1"/>
-<wire x1="12.065" y1="19.05" x2="14.605" y2="21.59" width="0.8128" layer="1"/>
-<wire x1="14.605" y1="21.59" x2="15.875" y2="21.59" width="0.8128" layer="1"/>
-<wire x1="1.27" y1="-5.08" x2="12.065" y2="5.715" width="0.8128" layer="1"/>
+<wire x1="11.43" y1="-4.445" x2="-6.35" y2="-4.445" width="0.6096" layer="1"/>
+<wire x1="-6.985" y1="-5.08" x2="-6.35" y2="-4.445" width="0.6096" layer="1"/>
+<wire x1="13.335" y1="-2.54" x2="13.335" y2="21.59" width="0.6096" layer="1"/>
+<wire x1="13.335" y1="21.59" x2="15.875" y2="21.59" width="0.6096" layer="1"/>
+<wire x1="11.43" y1="-4.445" x2="13.335" y2="-2.54" width="0.6096" layer="1"/>
 </signal>
 <signal name="SCL">
@@
 <wire x1="16.7728125" y1="19.05" x2="17.9340125" y2="20.2112" width="0.6096" layer="16"/>
 <wire x1="18.8959875" y1="20.2112" x2="20.0571875" y2="19.05" width="0.6096" layer="16"/>
-<wire x1="15.875" y1="19.05" x2="14.605" y2="19.05" width="0.8128" layer="1"/>
-<wire x1="14.605" y1="19.05" x2="13.97" y2="18.415" width="0.8128" layer="1"/>
-<wire x1="4.445" y1="-7.62" x2="1.905" y2="-10.16" width="0.8128" layer="1"/>
-<wire x1="1.905" y1="-10.16" x2="-3.81" y2="-10.16" width="0.8128" layer="1"/>
-<wire x1="-3.81" y1="-10.16" x2="-6.35" y2="-7.62" width="0.8128" layer="1"/>
-<wire x1="-6.35" y1="-7.62" x2="-6.985" y2="-7.62" width="0.8128" layer="1"/>
-<wire x1="4.445" y1="-4.445" x2="4.445" y2="-7.62" width="0.8128" layer="1"/>
-<wire x1="13.97" y1="5.08" x2="4.445" y2="-4.445" width="0.8128" layer="1"/>
-<wire x1="13.97" y1="18.415" x2="13.97" y2="5.08" width="0.8128" layer="1"/>
+<wire x1="15.875" y1="19.05" x2="15.24" y2="19.05" width="0.6096" layer="1"/>
+<wire x1="14.605" y1="18.415" x2="15.24" y2="19.05" width="0.6096" layer="1"/>
+<wire x1="-6.985" y1="-7.62" x2="-5.715" y2="-7.62" width="0.6096" layer="1"/>
+<wire x1="-5.715" y1="-7.62" x2="-3.175" y2="-10.16" width="0.6096" layer="1"/>
+<wire x1="-3.175" y1="-10.16" x2="2.54" y2="-10.16" width="0.6096" layer="1"/>
+<wire x1="2.54" y1="-10.16" x2="6.985" y2="-5.715" width="0.6096" layer="1"/>
+<wire x1="6.985" y1="-5.715" x2="12.7" y2="-5.715" width="0.6096" layer="1"/>
+<wire x1="12.7" y1="-5.715" x2="14.605" y2="-3.81" width="0.6096" layer="1"/>
+<wire x1="14.605" y1="-3.81" x2="14.605" y2="18.415" width="0.6096" layer="1"/>
 </signal>
 <signal name="SP+">
