File: pcb/OttoPi09-RPi3A-HAT/OttoPi09-RPi3A-HAT.brd (EAGLE design)
At the start: 56 x 65 mm, 40 parts

Commit message: UPD: pcb
Parts:
- removed DCDC1: (no value), ytani1:DCDC-MT3608-MOD1
- removed DCDC3: (no value), ytani1:DCDC-MT3608-MOD2-USB
- added NEOIN, PIND: (no value), ytani1:PINHEAD-MA01-1
- added NEOPIXEL: (no value), ytani1:PINHEAD-MA03-1
- added Q1: 2SK4017, ytani1:MOSFET-1
- added R6: 10K, rcl:0204/7
- added R7: 330, rcl:0204/7
- moved DCDC2 5.12 mm to (5.08, 6.35)
- moved SW2 1.27 mm to (-25.4, 6.35)
- moved GPIO 1.27 mm to (-25.4, 1.27)
- moved R1 1.27 mm to (-20.3, 16.5)
- renumbered AUDIO to AUD
Connections:
- net N$1 renamed GPIO10
- new net N$1: Q1.G, R6.1, R7.2
- new net N$2: NEOPIXEL.3, Q1.D
- new net N$5: PIND.1, R7.1
- new net N$8: NEOIN.1, NEOPIXEL.1
- net +5V: no longer DCDC1.VOUT+, DCDC3.VOUT+
- net BAT+: now also NEOPIXEL.2; no longer DCDC1.VIN+, DCDC3.VIN+
- net GND: now also Q1.S, R6.2; no longer DCDC1.VIN-, DCDC1.VOUT-, DCDC3.VIN-, DCDC3.VOUT-
Routing:
- net N$5: track 0.00 -> 7.77 mm
- net BAT+: track 118.9 -> 125.4 mm
- net N$1: track 0.00 -> 6.14 mm
- net N$2: track 0.00 -> 4.07 mm
- net +3V3: track 98.6 -> 95.0 mm
- net N$8: track 0.00 -> 2.54 mm
- net +5V: track 29.2 -> 27.1 mm
- net SDA: track 60.0 -> 61.3 mm
- net N$3: track 4.71 -> 3.81 mm
- net N$4: track 5.98 -> 5.08 mm
- net BAT+1: track 44.6 -> 45.3 mm
Other:
- board text added: "Q1"

Commit message: UPD: pcb
Parts:
- removed GPIO: (no value), ytani1:PINHEAD-MA01-1
- removed R2: 10K, rcl:0204/7
- removed SW2: (no value), ytani1:PINHEAD-MA02-1
- added IO4: (no value), ytani1:PINHEAD-MA01-1
- added LED2: (no value), led:LED3MM
- added OFF, ON: (no value), ytani1:PINHEAD-MA02-1
- added R8: 1K, rcl:0204/7
- moved Q1 6.35 mm to (10.8, 21.0), turned to 90 degrees
- moved R6 2.01 mm to (1.27, 19.7)
- moved R7 2.01 mm to (1.27, 22.2)
- moved ADC1 1.27 mm to (-8.89, 4.45)
- moved R1 1.27 mm to (-20.3, 17.8)
- moved LED1 0.64 mm to (-24.8, 14.0), turned to 180 degrees
- moved DCDC2 0.63 mm to (4.45, 6.35)
- moved R3 0.63 mm to (-20.3, 5.71)
- moved R4 0.63 mm to (-17.8, 5.71)
- moved R5 0.63 mm to (-15.2, 5.71)
- renumbered NEOIN to IO10, PIND to IO21
Connections:
- removed net N$4: GPIO.1, R2.1, SW2.2
- new net N$17: LED2.A, R8.1
- new net N$24: IO4.1, OFF.2
- net +3V3: no longer R2.2
- net GND: now also LED2.K, OFF.1, ON.1; no longer SW2.1
- net N$5: now also R8.2
- net SCL: now also ON.2
Routing:
- net SCL: track 58.3 -> 86.2 mm
- net GND: track 0.00 -> 23.8 mm
- net +3V3: track 95.0 -> 82.4 mm
- net N$17: track 0.00 -> 7.67 mm
- net BAT+: track 125.4 -> 131.8 mm, vias 2 -> 0
- net N$2: track 4.07 -> 10.1 mm
- net N$4: track 5.08 -> 0.00 mm
- net N$24: track 0.00 -> 2.54 mm
- net +5V: track 27.1 -> 29.6 mm
- net N$1: track 6.14 -> 8.35 mm
- net SDA: track 61.3 -> 60.3 mm
- net N$26: track 5.34 -> 6.35 mm
- net BAT+1: track 45.3 -> 44.6 mm
- net N$3: track 3.81 -> 3.18 mm
- net N$15: track 18.8 -> 18.2 mm

Commit message: UPD: pcb
Parts:
- added BAT0: BAT0+, ytani1:PINHEAD-MA02-1
- BAT0+: value BAT1 -> (none)
- moved DCDC2 2.29 mm to (5.71, 8.26)
- moved Q1 1.80 mm to (9.53, 22.2)
- moved R6 1.27 mm to (1.27, 21.0)
- moved R7 1.27 mm to (1.27, 23.5)
- moved R8 1.27 mm to (1.27, 26.0)
- moved CHG1 0.64 mm to (5.08, -19.6)
- turned BAT+ to 270 degrees
- turned JP1 to 90 degrees
Connections:
- net BAT+0: now also BAT0.1
- net BAT-0: now also BAT0.2
Routing:
- net BAT+: track 131.8 -> 139.2 mm
- net BAT-0: track 26.4 -> 33.5 mm
- net +5V: track 29.6 -> 33.1 mm
- net BAT+2: track 12.2 -> 8.94 mm
- net +3V3: track 82.4 -> 85.6 mm
- net BAT+0: track 32.4 -> 35.0 mm
- net N$2: track 10.1 -> 7.88 mm
- net BAT+1: track 44.6 -> 46.4 mm
- net N$5: track 7.62 -> 6.35 mm
- net N$1: track 8.35 -> 7.08 mm
- net SCL: track 86.2 -> 87.4 mm
- net N$15: track 18.2 -> 19.4 mm
- net SDA: track 60.3 -> 61.1 mm
- net SP-: track 5.87 -> 5.13 mm
- net GND: track 23.8 -> 24.4 mm
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