File: pcb/OttoPi09-RPi3A-HAT/OttoPi09-RPi3A-HAT.sch (EAGLE design)
At the start: 40 parts

Commit message: UPD: pcb
Parts:
- removed DCDC1: (no value), ytani1:DCDC-MT3608-MOD
- removed DCDC3: (no value), ytani1:DCDC-MT3608-MODUSB
- added NEOIN, PIND: (no value), ytani1:PINHEAD-MA01-1
- added NEOPIXEL: (no value), ytani1:PINHEAD-MA03-1
- added Q1: 2SK4017, ytani1:MOSFET-2SK4017
- added R6: 10K, rcl:R-US_0204/7
- added R7: 330, rcl:R-US_0204/7
- renumbered AUDIO to AUD
Connections:
- net N$1 renamed GPIO10
- new net N$1: Q1.G, R6.1, R7.2
- new net N$2: NEOPIXEL.3, Q1.D
- new net N$5: PIND.1, R7.1
- new net N$8: NEOIN.1, NEOPIXEL.1
- net +5V: no longer DCDC1.VOUT+, DCDC3.VOUT+
- net BAT+: now also NEOPIXEL.2; no longer DCDC1.VIN+, DCDC3.VIN+
- net GND: now also Q1.S, R6.2; no longer DCDC1.VIN-, DCDC1.VOUT-, DCDC3.VIN-, DCDC3.VOUT-
Other:
- moved on the sheet: ADC1, R3, R4, R5

Commit message: UPD: pcb
Parts:
- removed GPIO: (no value), ytani1:PINHEAD-MA01-1
- removed R2: 10K, rcl:R-US_0204/7
- removed SW2: (no value), ytani1:PINHEAD-MA02-1
- added IO4: (no value), ytani1:PINHEAD-MA01-1
- added LED2: (no value), led:LED3MM
- added OFF, ON: (no value), ytani1:PINHEAD-MA02-1
- added R8: 1K, rcl:R-US_0204/7
- renumbered NEOIN to IO10, PIND to IO21
Connections:
- removed net N$4: GPIO.1, R2.1, SW2.2
- new net N$17: LED2.A, R8.1
- new net N$24: IO4.1, OFF.2
- net +3V3: no longer R2.2
- net GND: now also LED2.C, OFF.1, ON.1; no longer SW2.1
- net N$5: now also R8.2
- net SCL: now also ON.2

Commit message: UPD: pcb
Parts:
- added BAT0: BAT0+, ytani1:PINHEAD-MA02-1
- BAT0+: value BAT1 -> (none)
Connections:
- net BAT+0: now also BAT0.1
- net BAT-0: now also BAT0.2
Other:
- moved on the sheet: +5V, BAT+, BAT0+, CHG1, DCDC2, JP1, LED1, R1, SW1
